File: HPS_Round_Clock/HPS_Round_Clock.kicad_sch (KiCad schematic)
At the start: 15 parts

Commit message: Update HPS_Round_Clock.kicad_sch
Parts:
- removed C?: C_0805_10uf, footprints:C_0805_2012Metric, symbol HPS:C_0805_10uf
- removed D?: LED_0805, footprints:LED_0805_2012Metric, symbol HPS:LED_0805
- removed H1, H2, H3, H4: MountingHole, footprints:MountingHole_3.2mm_M3, symbol HPS:MountingHole
- removed J?: Conn_01x06, footprints:PinHeader_1x06_P2.54mm_Vertical, symbol HPS:Conn_01x06
- removed R?: R_0805_2.2K, footprints:R_0805_2012Metric, symbol HPS:R_0805_2.2K
- added C3, C7: C_0805_0.1uf, footprints:C_0805_2012Metric, symbol HPS:C_0805_0.1uf
- added C6: C_0805_1uf, footprints:C_0805_2012Metric, symbol HPS:C_0805_1uf
- added D1: LED_0805, footprints:LED_0805_2012Metric, symbol HPS:LED_0805
- added J1: Conn_01x06, footprints:PinHeader_1x06_P2.54mm_Vertical, symbol HPS:Conn_01x06
- added J2: PJ-102AH, footprints:PJ-102AH, symbol HPS:PJ-102AH
- added R1: R_0805_2.2K, footprints:R_0805_2012Metric, symbol HPS:R_0805_2.2K
- added R3, R4: R_0805_47, footprints:R_0805_2012Metric, symbol HPS:R_0805_47
- added SW1: Omron_B3F_SPST, footprints:SW_SPST_Omron_B3FS-100xP, symbol HPS:Omron_B3F_SPST
- added U2: L7805, symbol HPS:L7805
- gave numbers to parts that had none: 7
Connections:
- net GND: now also C6.2, C7.2, J1.1 (Pin_1), J1.2 (Pin_2), J2.2 (OUT), R1.2, SW1.1 (A), SW1.2 (A), U2.2 (GND)
- net LED_SCK: now also D1.2 (A)
- net RESET: now also C3.2, SW1.3 (B), SW1.4 (B)
- net VCC: now also C7.1, U2.3 (OUT)
- net PD0 renamed RXD
- net RXD: now also R3.2
- net PD1 renamed TXD
- net TXD: now also R4.2
- net XTAL1: no longer names the net of C4.2, U1.9 (XTAL1/PB6), Y1.2
- net XTAL2: no longer names the net of C5.2, U1.10 (XTAL2/PB7), Y1.1
- new net: C6.1, J2.1 (POLE), U2.1 (IN)
- new net: C3.1, J1.6 (Pin_6)
- new net: D1.1 (K), R1.1
- new net: J1.4 (Pin_4), R4.1
- new net: J1.5 (Pin_5), R3.1
- no-connect marks 1 -> 2
Other:
- moved on the sheet: C1, C2, C4, C5, R2, U1, Y1

Commit message: Update HPS_Round_Clock.kicad_sch
Other:
- note added: "LED"
- note added: "MCU"
- note added: "Power Input"
- note added: "Serial"
Changed lines of the file:
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@@
     (stroke (width 0) (type default) (color 0 0 0 0))
   )
-  (label "Serial" (at 134.62 189.23 0)
-    (effects (font (size 3 3) (thickness 0.6) bold) (justify left bottom))
+  (text "MCU" (at 133.35 121.92 0)
+    (effects (font (size 5 5) (thickness 1) bold) (justify left bottom))
   )
-  (label "LED" (at 49.53 189.23 0)
+  (text "Serial" (at 134.62 189.23 0)
     (effects (font (size 3 3) bold) (justify left bottom))
   )
-  (label "Power Input" (at 238.76 74.93 0)
+  (text "Power Input" (at 238.76 74.93 0)
     (effects (font (size 3 3) bold) (justify left bottom))
   )
-  (label "MCU" (at 133.35 121.92 0)
-    (effects (font (size 5 5) (thickness 1) bold) (justify left bottom))
+  (text "LED" (at 49.53 189.23 0)
+    (effects (font (size 3 3) bold) (justify left bottom))
   )
   (global_label "LED_SCK" (shape input) (at 33.02 146.05 90) (fields_autoplaced)
