File: HPS_Round_Clock/HPS_Round_Clock.kicad_sch (KiCad schematic)
At the start: 18 parts, among them J1 Conn_01x06, J2 PJ-102AH, SW1 Omron_B3F_SPST, U1 ATmega328-PU, U2 L7805, Y1 Crystal_16MHz

Commit message: Update HPS_Round_Clock.kicad_sch
Parts:
- added D? (x72): NEOPIXEL_THT, footprints:Adafruit_Neopixel_TH_1938, symbol HPS:NEOPIXEL_THT
- added DS1: LED_Display_1001, footprints:Adafruit-1001-0-0-MFG, symbol HPS:LED_Display_1001
- added R5, R6, R7, R8, R?: R_0805_10K, footprints:R_0805_2012Metric, symbol HPS:R_0805_10K
- added SW1, SW2, SW3, SW4: Omron_B3F_SPST, footprints:SW_SPST_Omron_B3FS-100xP, symbol HPS:Omron_B3F_SPST
- added U2: MAX7219, footprints:DIP-24_W7.62mm, symbol HPS:MAX7219
Connections:
- net GND: now also D?.1 (VSS), D?.1 (VSS), D?.1 (VSS), D?.1 (VSS), D?.1 (VSS), D?.1 (VSS), D?.1 (VSS), D?.1 (VSS), D?.1 (VSS), D?.1 (VSS), D?.1 (VSS), D?.1 (VSS), D?.1 (VSS), D?.1 (VSS), D?.1 (VSS), D?.1 (VSS), D?.1 (VSS), D?.1 (VSS), D?.1 (VSS), D?.1 (VSS), D?.1 (VSS), D?.1 (VSS), D?.1 (VSS), D?.1 (VSS), D?.1 (VSS), D?.1 (VSS), D?.1 (VSS), D?.1 (VSS), D?.1 (VSS), D?.1 (VSS), D?.1 (VSS), D?.1 (VSS), D?.1 (VSS), D?.1 (VSS), D?.1 (VSS), D?.1 (VSS), D?.1 (VSS), D?.1 (VSS), D?.1 (VSS), D?.1 (VSS), D?.1 (VSS), D?.1 (VSS), D?.1 (VSS), D?.1 (VSS), D?.1 (VSS), D?.1 (VSS), D?.1 (VSS), D?.1 (VSS), D?.1 (VSS), D?.1 (VSS), D?.1 (VSS), D?.1 (VSS), D?.1 (VSS), D?.1 (VSS), D?.1 (VSS), D?.1 (VSS), D?.1 (VSS), D?.1 (VSS), D?.1 (VSS), D?.1 (VSS), D?.1 (VSS), D?.1 (VSS), D?.1 (VSS), D?.1 (VSS), D?.1 (VSS), D?.1 (VSS), D?.1 (VSS), D?.1 (VSS), D?.1 (VSS), D?.1 (VSS), D?.1 (VSS), D?.1 (VSS), R5.1, R6.1, R7.1, R8.1, U2.4 (GND), U2.9 (GND)
- net LED_SCK: no longer U1.19 (PB5)
- net VCC: now also D?.3 (VDD), D?.3 (VDD), D?.3 (VDD), D?.3 (VDD), D?.3 (VDD), D?.3 (VDD), D?.3 (VDD), D?.3 (VDD), D?.3 (VDD), D?.3 (VDD), D?.3 (VDD), D?.3 (VDD), D?.3 (VDD), D?.3 (VDD), D?.3 (VDD), D?.3 (VDD), D?.3 (VDD), D?.3 (VDD), D?.3 (VDD), D?.3 (VDD), D?.3 (VDD), D?.3 (VDD), D?.3 (VDD), D?.3 (VDD), D?.3 (VDD), D?.3 (VDD), D?.3 (VDD), D?.3 (VDD), D?.3 (VDD), D?.3 (VDD), D?.3 (VDD), D?.3 (VDD), D?.3 (VDD), D?.3 (VDD), D?.3 (VDD), D?.3 (VDD), D?.3 (VDD), D?.3 (VDD), D?.3 (VDD), D?.3 (VDD), D?.3 (VDD), D?.3 (VDD), D?.3 (VDD), D?.3 (VDD), D?.3 (VDD), D?.3 (VDD), D?.3 (VDD), D?.3 (VDD), D?.3 (VDD), D?.3 (VDD), D?.3 (VDD), D?.3 (VDD), D?.3 (VDD), D?.3 (VDD), D?.3 (VDD), D?.3 (VDD), D?.3 (VDD), D?.3 (VDD), D?.3 (VDD), D?.3 (VDD), D?.3 (VDD), D?.3 (VDD), D?.3 (VDD), D?.3 (VDD), D?.3 (VDD), D?.3 (VDD), D?.3 (VDD), D?.3 (VDD), D?.3 (VDD), D?.3 (VDD), D?.3 (VDD), D?.3 (VDD), R?.1, SW1.4 (B), SW2.4 (B), SW3.4 (B), SW4.4 (B), U2.19 (V+)
- net Button (Brightness): no longer names the net of U1.5 (PD3)
- net Button (Brightness): now also SW1.1 (A)
- net Button (Color): no longer names the net of U1.6 (PD4)
- net Button (Color): now also SW2.1 (A)
- net Button (Hours): no longer names the net of U1.13 (PD7)
- net Button (Hours): now also SW3.1 (A)
- net Button (Minutes): no longer names the net of U1.14 (PB0)
- net Button (Minutes): now also SW4.1 (A)
- net MAX 7219 MISO renamed IR Module MISO
- new net: R6.2, SW3.3 (B)
- new net: D?.2 (DIN), D?.4 (DOUT) (x70)
- new net: R7.2, SW4.3 (B)
- new net: R?.2, U2.18 (ISET)
- new net: R8.2, SW1.3 (B)
- new net: R5.2, SW2.3 (B)
- new net: DS1.11 (COM_DIG.2), U2.11 (DIG_1)
- new net: DS1.13 (A), U2.14 (SEG_A)
- new net: DS1.12 (F), U2.15 (SEG_F)
- new net: DS1.9 (B), U2.16 (SEG_B)
- new net: DS1.5 (G), U2.17 (SEG_G)
- new net: DS1.14 (COM_DIG.1), U2.2 (DIG_0)
- new net: DS1.4 (C), U2.20 (SEG_C)
- new net: DS1.1 (E), U2.21 (SEG_E)
- new net: DS1.3 (DP), U2.22 (SEG_DP)
- new net: DS1.2 (D), U2.23 (SEG_D)
- new net: DS1.10 (COM_DIG.3), U2.6 (DIG_2)
- new net: DS1.6 (COM_DIG.4), U2.7 (DIG_3)
- new net MAX 7219 SCK: U1.19 (PB5)
- new net MCU MOSI: U2.1 (DIN)
- new net MCU PD5: D?.2 (DIN), D?.2 (DIN)
- new net MCU SCK: U2.13 (CLK)
- new net MCU SS: U2.12 (LOAD)
- no-connect marks 2 -> 18
Other:
- note added: "Button (Brightness)"
- note added: "Button (Color)"
- note added: "Button (Hours)"
- note added: "Button (Minutes)"
- note added: "Inner LED Ring"
- note added: "MAX 7219 & LED Display"
- note added: "Outer LED Ring"
- moved on the sheet: C1, C2, C3, C4, C5, C6, C7, D1, J1, J2, R1, R2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

Commit message: Update HPS_Round_Clock.kicad_sch
Parts:
- removed D1: LED_0805, footprints:LED_0805_2012Metric, symbol HPS:LED_0805
- removed D? (x12): NEOPIXEL_THT, footprints:Adafruit_Neopixel_TH_1938, symbol HPS:NEOPIXEL_THT
- removed R1: R_0805_2.2K, footprints:R_0805_2012Metric, symbol HPS:R_0805_2.2K
- added C8, C9 (x2): C_0805_0.1uf, footprints:C_0805_2012Metric, symbol HPS:C_0805_0.1uf
- gave numbers to parts that had none: 61
- renumbered C2 to C1, C6 to C2, C7 to C3, C1 to C5, C5 to C6, C3 to C7, J2 to J1, J1 to J2, R7 to R1, R8 to R3, R5 to R4, R6 to R5, R3 to R6, R4 to R7, SW4 to SW1, SW1 to SW2, SW2 to SW3, SW3 to SW4, SW1 to SW5, U2 to U1, U1 to U2, U2 to U3
Connections:
- net MCU MOSI is gone; now on net MOSI: U3.1 (DIN)
- net MCU SCK is gone; now on net SCK: U3.13 (CLK)
- net MCU SS is gone; now on net SS: U3.12 (LOAD)
- net GND: now also C8.2, C9.2, C9.2
- net Inner LED Ring: now also D61.2 (DIN)
- net Outer LED Ring: now also D1.2 (DIN)
- net VCC: now also C8.1, C9.1, C9.1
- net MAX 7219 MOSI renamed MOSI
- net MAX 7219 SCK renamed SCK
- net MAX 7219 SS renamed SS
- removed net MCU PD5: D1.2 (DIN), D61.2 (DIN)
- net RTC SCL renamed SCL
- net RTC SDA renamed SDA
Other:
- note removed: "LED"
- moved on the sheet: C7, J2, R6, R7, SW5

Commit message: Update HPS_Round_Clock.kicad_sch
Parts:
- removed D31, D32, D33, D34, D57, D58, D59, D60: NEOPIXEL_THT, footprints:Adafruit_Neopixel_TH_1938, symbol HPS:NEOPIXEL_THT
- added BT1: Battery_Cell, footprints:BatteryHolder_Keystone_106_1x20mm, symbol HPS:Battery_Cell
- added C10, C11, C13, C15, C16, C9: C_0805_0.1uf, footprints:C_0805_2012Metric, symbol HPS:C_0805_0.1uf
- added D21, D22, D23, D24, D41, D42, D43, D44, D45, D46, D47, D48, D61, D62, D63, D64, D69, D70, D71, D72: NEOPIXEL_THT, footprints:Adafruit_Neopixel_TH_1938, symbol HPS:NEOPIXEL_THT
- added U2: DS1307_DIP-8, footprints:DIP-8_W7.62mm, symbol HPS:DS1307_DIP-8
- renumbered C9 to C12, C9 to C14, D39 to D31, D40 to D32, D41 to D33, D42 to D34, D43 to D35, D44 to D36, D45 to D37, D46 to D38, D47 to D39, D48 to D40, D61 to D49, D62 to D50, D63 to D51, D64 to D52, D69 to D57, D70 to D58, D71 to D59, D72 to D60, U2 to U4
Connections:
- net GND: now also BT1.2 (-), C10.2, C11.2, C13.2, C15.2, C16.2, C9.2, D21.1 (VSS), D22.1 (VSS), D23.1 (VSS), D24.1 (VSS), D41.1 (VSS), D42.1 (VSS), D43.1 (VSS), D44.1 (VSS), D45.1 (VSS), D46.1 (VSS), D47.1 (VSS), D48.1 (VSS), D61.1 (VSS), D62.1 (VSS), D63.1 (VSS), D64.1 (VSS), D69.1 (VSS), D70.1 (VSS), D71.1 (VSS), D72.1 (VSS), U2.4 (GND); no longer C4.1, C6.1
- net SCL: now also U2.6 (SCL)
- net SDA: now also U2.5 (SDA)
- net VCC: now also SW1.3 (B), SW2.3 (B), SW3.3 (B), SW4.3 (B), BT1.1 (+), C10.1, C11.1, C13.1, C15.1, C16.1, C9.1, D21.3 (VDD), D22.3 (VDD), D23.3 (VDD), D24.3 (VDD), D41.3 (VDD), D42.3 (VDD), D43.3 (VDD), D44.3 (VDD), D45.3 (VDD), D46.3 (VDD), D47.3 (VDD), D48.3 (VDD), D61.3 (VDD), D62.3 (VDD), D63.3 (VDD), D64.3 (VDD), D69.3 (VDD), D70.3 (VDD), D71.3 (VDD), D72.3 (VDD), U2.3 (VBAT), U2.8 (VCC); no longer SW1.4 (B), SW2.4 (B), SW3.4 (B), SW4.4 (B)
- net at R5.2: now also SW4.1 (A), U4.13 (PD7); no longer SW4.3 (B)
- net at R1.2: now also SW1.1 (A), U4.14 (PB0); no longer SW1.3 (B)
- net at D56.4 (DOUT): now also D57.2 (DIN)
- net at D52.4 (DOUT): now also D53.2 (DIN); no longer D65.2 (DIN)
- net at R3.2: now also SW2.1 (A), U4.5 (PD3); no longer SW2.3 (B)
- net at D30.4 (DOUT): now also D31.2 (DIN)
- net at D68.4 (DOUT): now also D69.2 (DIN); no longer D57.2 (DIN)
- net at R4.2: now also SW3.1 (A), U4.6 (PD4); no longer SW3.3 (B)
- net at D40.4 (DOUT): now also D41.2 (DIN); no longer D53.2 (DIN)
- net at D20.4 (DOUT): now also D21.2 (DIN); no longer D25.2 (DIN)
- net IR Module MISO: no longer names the net of U4.18 (PB4)
- net IR Reciever: no longer names the net of U4.4 (PD2)
- new net: C6.1, U2.2 (X2)
- new net: D21.4 (DOUT), D22.2 (DIN)
- new net: D43.4 (DOUT), D44.2 (DIN)
- new net: D44.4 (DOUT), D45.2 (DIN)
- new net: C4.1, U2.1 (X1)
- new net: D48.4 (DOUT), D61.2 (DIN)
- new net: D61.4 (DOUT), D62.2 (DIN)
- new net: D42.4 (DOUT), D43.2 (DIN)
- new net: D46.4 (DOUT), D47.2 (DIN)
- new net: D47.4 (DOUT), D48.2 (DIN)
- new net: D23.4 (DOUT), D24.2 (DIN)
- new net: D24.4 (DOUT), D25.2 (DIN)
- new net: D41.4 (DOUT), D42.2 (DIN)
- new net: D45.4 (DOUT), D46.2 (DIN)
- new net: D70.4 (DOUT), D71.2 (DIN)
- new net: D71.4 (DOUT), D72.2 (DIN)
- new net: D69.4 (DOUT), D70.2 (DIN)
- new net: D63.4 (DOUT), D64.2 (DIN)
- new net: D64.4 (DOUT), D65.2 (DIN)
- new net: D62.4 (DOUT), D63.2 (DIN)
- new net: D22.4 (DOUT), D23.2 (DIN)
- no-connect marks 18 -> 27
Other:
- note added: "IR Module MISO"
- note added: "IR Receiver"
- moved on the sheet: C2, C3, C7, D49, D50, D51, D52, D57, D58, D59, D60, DS1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

Commit message: Update HPS_Round_Clock.kicad_sch
Parts:
- added D73: LED_0805, footprints:LED_0805_2012Metric, symbol HPS:LED_0805
- added R9: R_0805_1K, footprints:R_0805_2012Metric, symbol HPS:R_0805_1K
- added U5: TSOP38238, footprints:Vishay_MINICAST-3Pin, symbol HPS:TSOP38238
- added Y2: Crystal_32768Hz, footprints:Crystal_SMD_2Pin_3.2x1.5mm, symbol HPS:Crystal_32768Hz
- renumbered C8 to C61, C9 to C62, C10 to C63, D61 to D49, D62 to D50, D63 to D51, D64 to D52, D65 to D53, D66 to D54, D67 to D55, D68 to D56, D69 to D57, D70 to D58, D71 to D59, D72 to D60, D49 to D61, D50 to D62, D51 to D63, D52 to D64, D53 to D65, D54 to D66, D55 to D67, D56 to D68, D57 to D69, D58 to D70, D59 to D71, D60 to D72
Connections:
- net GND: now also C4.1, C6.1, U5.2 (GND)
- net Inner LED Ring: no longer D61.2 (DIN)
- net VCC: now also D73.2 (A), U5.3 (Vs); no longer BT1.1 (+), U2.3 (VBAT)
- net at U2.2 (X2): now also Y2.2; no longer C6.1
- net at U2.1 (X1): now also Y2.1; no longer C4.1
- net LEDs: now reaches D60.4 (DOUT)
- net LEDs: now also D61.2 (DIN)
- net IR Receiver: now reaches U4.4 (PD2)
- net IR Receiver: now also R9.1, U5.1 (OUT)
- new net: BT1.1 (+), U2.3 (VBAT)
- new net: D73.1 (K), R9.2
- no-connect marks 27 -> 25
Other:
- note added: "RTC"
- note removed: "IR Module MISO"
- moved on the sheet: BT1, C61, C62, C63, C7, D61, D62, D63, D64, D65, D66, D67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

Commit message: Update HPS_Round_Clock.kicad_sch
Parts:
- removed C16, C61, C62, C63: C_0805_0.1uf, footprints:C_0805_2012Metric, symbol HPS:C_0805_0.1uf
- removed D1, D10, D11, D12, D13, D14, D15, D16, D17, D18, D19, D2, D20, D21, D22, D23, D24, D25, D26, D27, D28, D29, D3, D30, D31, D32, D33, D34, D35, D36, D37, D38, D39, D4, D40, D41, D42, D43, D44, D45, D46, D47, D48, D49, D5, D50, D51, D52, D53, D54, D55, D56, D57, D58, D59, D6, D60, D61, D62, D63, D64, D65, D66, D67, D68, D69, D7, D70, D71, D72, D8, D9: NEOPIXEL_THT, footprints:Adafruit_Neopixel_TH_1938, symbol HPS:NEOPIXEL_THT
- added C13, C14, C15: C_0805_0.1uf, footprints:C_0805_2012Metric, symbol HPS:C_0805_0.1uf
- added D1, D10, D11, D12, D13, D14, D15, D16, D17, D18, D19, D2, D20, D21, D22, D23, D24, D25, D26, D27, D28, D29, D3, D30, D31, D32, D33, D34, D35, D36, D37, D38, D39, D4, D40, D41, D42, D43, D44, D45, D46, D47, D48, D49, D5, D50, D51, D52, D53, D54, D55, D56, D57, D58, D59, D6, D60, D61, D62, D63, D64, D65, D66, D67, D68, D69, D7, D70, D71, D72, D8, D9: NEOPIXEL_SMT, footprints:LED_SK6812_PLCC4_5.0x5.0mm_P3.2mm, symbol HPS:NEOPIXEL_SMT
- renumbered C13 to C10, C14 to C11, C15 to C12, C11 to C8, C12 to C9
Connections:
- net GND: now also C13.2, C14.2, C15.2, D1.1 (VSS), D10.1 (VSS), D11.1 (VSS), D12.1 (VSS), D13.1 (VSS), D14.1 (VSS), D15.1 (VSS), D16.1 (VSS), D17.1 (VSS), D18.1 (VSS), D19.1 (VSS), D2.1 (VSS), D20.1 (VSS), D21.1 (VSS), D22.1 (VSS), D23.1 (VSS), D24.1 (VSS), D25.1 (VSS), D26.1 (VSS), D27.1 (VSS), D28.1 (VSS), D29.1 (VSS), D3.1 (VSS), D30.1 (VSS), D31.1 (VSS), D32.1 (VSS), D33.1 (VSS), D34.1 (VSS), D35.1 (VSS), D36.1 (VSS), D37.1 (VSS), D38.1 (VSS), D39.1 (VSS), D4.1 (VSS), D40.1 (VSS), D41.1 (VSS), D42.1 (VSS), D43.1 (VSS), D44.1 (VSS), D45.1 (VSS), D46.1 (VSS), D47.1 (VSS), D48.1 (VSS), D49.1 (VSS), D5.1 (VSS), D50.1 (VSS), D51.1 (VSS), D52.1 (VSS), D53.1 (VSS), D54.1 (VSS), D55.1 (VSS), D56.1 (VSS), D57.1 (VSS), D58.1 (VSS), D59.1 (VSS), D6.1 (VSS), D60.1 (VSS), D61.1 (VSS), D62.1 (VSS), D63.1 (VSS), D64.1 (VSS), D65.1 (VSS), D66.1 (VSS), D67.1 (VSS), D68.1 (VSS), D69.1 (VSS), D7.1 (VSS), D70.1 (VSS), D71.1 (VSS), D72.1 (VSS), D8.1 (VSS), D9.1 (VSS)
- net Outer LED Ring: now also D1.2 (DIN)
- net VCC: now also C13.1, C14.1, C15.1, D1.3 (VDD), D10.3 (VDD), D11.3 (VDD), D12.3 (VDD), D13.3 (VDD), D14.3 (VDD), D15.3 (VDD), D16.3 (VDD), D17.3 (VDD), D18.3 (VDD), D19.3 (VDD), D2.3 (VDD), D20.3 (VDD), D21.3 (VDD), D22.3 (VDD), D23.3 (VDD), D24.3 (VDD), D25.3 (VDD), D26.3 (VDD), D27.3 (VDD), D28.3 (VDD), D29.3 (VDD), D3.3 (VDD), D30.3 (VDD), D31.3 (VDD), D32.3 (VDD), D33.3 (VDD), D34.3 (VDD), D35.3 (VDD), D36.3 (VDD), D37.3 (VDD), D38.3 (VDD), D39.3 (VDD), D4.3 (VDD), D40.3 (VDD), D41.3 (VDD), D42.3 (VDD), D43.3 (VDD), D44.3 (VDD), D45.3 (VDD), D46.3 (VDD), D47.3 (VDD), D48.3 (VDD), D49.3 (VDD), D5.3 (VDD), D50.3 (VDD), D51.3 (VDD), D52.3 (VDD), D53.3 (VDD), D54.3 (VDD), D55.3 (VDD), D56.3 (VDD), D57.3 (VDD), D58.3 (VDD), D59.3 (VDD), D6.3 (VDD), D60.3 (VDD), D61.3 (VDD), D62.3 (VDD), D63.3 (VDD), D64.3 (VDD), D65.3 (VDD), D66.3 (VDD), D67.3 (VDD), D68.3 (VDD), D69.3 (VDD), D7.3 (VDD), D70.3 (VDD), D71.3 (VDD), D72.3 (VDD), D8.3 (VDD), D9.3 (VDD)
- net Inner LED Ring: no longer names the net of U4.11 (PD5)
- new net: D52.4 (DOUT), D53.2 (DIN)
- new net: D53.4 (DOUT), D54.2 (DIN)
- new net: D44.4 (DOUT), D45.2 (DIN)
- new net: D45.4 (DOUT), D46.2 (DIN)
- new net: D32.4 (DOUT), D33.2 (DIN)
- new net: D33.4 (DOUT), D34.2 (DIN)
- new net: D20.4 (DOUT), D21.2 (DIN)
- new net: D21.4 (DOUT), D22.2 (DIN)
- new net: D69.4 (DOUT), D70.2 (DIN)
- new net: D70.4 (DOUT), D71.2 (DIN)
- new net: D17.4 (DOUT), D18.2 (DIN)
- new net: D18.4 (DOUT), D19.2 (DIN)
- new net: D19.4 (DOUT), D20.2 (DIN)
- new net: D71.4 (DOUT), D72.2 (DIN)
- new net: D10.4 (DOUT), D11.2 (DIN)
- new net: D11.4 (DOUT), D12.2 (DIN)
- new net: D1.4 (DOUT), D2.2 (DIN)
- new net: D2.4 (DOUT), D3.2 (DIN)
- new net: D12.4 (DOUT), D13.2 (DIN)
- new net: D25.4 (DOUT), D26.2 (DIN)
- new net: D26.4 (DOUT), D27.2 (DIN)
- new net: D54.4 (DOUT), D55.2 (DIN)
- new net: D41.4 (DOUT), D42.2 (DIN)
- new net: D42.4 (DOUT), D43.2 (DIN)
- new net: D35.4 (DOUT), D36.2 (DIN)
- new net: D36.4 (DOUT), D37.2 (DIN)
- new net: D27.4 (DOUT), D28.2 (DIN)
- new net: D28.4 (DOUT), D29.2 (DIN)
- new net: D5.4 (DOUT), D6.2 (DIN)
- new net: D6.4 (DOUT), D7.2 (DIN)
- new net: D7.4 (DOUT), D8.2 (DIN)
- new net: D8.4 (DOUT), D9.2 (DIN)
- new net: D13.4 (DOUT), D14.2 (DIN)
- new net: D56.4 (DOUT), D57.2 (DIN)
- new net: D57.4 (DOUT), D58.2 (DIN)
- new net: D10.2 (DIN), D9.4 (DOUT)
- new net: D43.4 (DOUT), D44.2 (DIN)
- new net: D66.4 (DOUT), D67.2 (DIN)
- new net: D67.4 (DOUT), D68.2 (DIN)
- new net: D3.4 (DOUT), D4.2 (DIN)
- new net: D30.4 (DOUT), D31.2 (DIN)
- new net: D31.4 (DOUT), D32.2 (DIN)
- new net: D46.4 (DOUT), D47.2 (DIN)
- new net: D47.4 (DOUT), D48.2 (DIN)
- new net: D22.4 (DOUT), D23.2 (DIN)
- new net: D23.4 (DOUT), D24.2 (DIN)
- new net: D62.4 (DOUT), D63.2 (DIN)
- new net: D63.4 (DOUT), D64.2 (DIN)
- new net: D14.4 (DOUT), D15.2 (DIN)
- new net: D48.4 (DOUT), D49.2 (DIN)
- new net: D38.4 (DOUT), D39.2 (DIN)
- new net: D39.4 (DOUT), D40.2 (DIN)
- new net: D55.4 (DOUT), D56.2 (DIN)
- new net: D4.4 (DOUT), D5.2 (DIN)
- new net: D15.4 (DOUT), D16.2 (DIN)
- new net: D16.4 (DOUT), D17.2 (DIN)
- new net: D58.4 (DOUT), D59.2 (DIN)
- new net: D24.4 (DOUT), D25.2 (DIN)
- new net: D59.4 (DOUT), D60.2 (DIN)
- new net: D65.4 (DOUT), D66.2 (DIN)
- new net: D60.4 (DOUT), D61.2 (DIN)
- new net: D68.4 (DOUT), D69.2 (DIN)
- new net: D34.4 (DOUT), D35.2 (DIN)
- new net: D40.4 (DOUT), D41.2 (DIN)
- new net: D61.4 (DOUT), D62.2 (DIN)
- new net: D64.4 (DOUT), D65.2 (DIN)
- new net: D49.4 (DOUT), D50.2 (DIN)
- new net: D50.4 (DOUT), D51.2 (DIN)
- new net: D29.4 (DOUT), D30.2 (DIN)
- new net: D51.4 (DOUT), D52.2 (DIN)
- new net: D37.4 (DOUT), D38.2 (DIN)
- no-connect marks 25 -> 26
Other:
- note added: "LED Ring"
- note removed: "Inner LED Ring"
- note removed: "Outer LED Ring"
- moved on the sheet: C10, C11, C12, C8, C9

Commit message: Update HPS_Round_Clock.kicad_sch
Parts:
- removed C14, C15: C_0805_0.1uf, footprints:C_0805_2012Metric, symbol HPS:C_0805_0.1uf
- removed D61, D62, D63, D64, D65, D66, D67, D68, D69, D70, D71, D72: NEOPIXEL_SMT, footprints:LED_SK6812_PLCC4_5.0x5.0mm_P3.2mm, symbol HPS:NEOPIXEL_SMT

Commit message: Update HPS_Round_Clock.kicad_sch
Parts:
- removed C13: C_0805_0.1uf, footprints:C_0805_2012Metric, symbol HPS:C_0805_0.1uf
- removed D46, D47, D48, D49, D50, D51, D52, D53, D54, D55, D56, D57, D58, D59, D60: NEOPIXEL_SMT, footprints:LED_SK6812_PLCC4_5.0x5.0mm_P3.2mm, symbol HPS:NEOPIXEL_SMT
- removed DS1: LED_Display_1001, footprints:Adafruit-1001-0-0-MFG, symbol HPS:LED_Display_1001
- removed J1: PJ-102AH, footprints:PJ-102AH, symbol HPS:PJ-102AH
- removed R8: R_0805_10K, footprints:R_0805_2012Metric, symbol HPS:R_0805_10K
- removed U3: MAX7219, footprints:DIP-24_W7.62mm, symbol HPS:MAX7219
- added J1: Power_inlet_vertical, footprints:Wurth-694106402002, symbol HPS:Power_inlet_vertical
- U1: footprint (none) -> footprints:TO-252-2; Digikey PN (none) -> 497-7255-1-ND; MFG (none) -> STMicroelectronics; MPN (none) -> L7805CDT-TR
- renumbered D73 to D100
Connections:
- net GND: now also J1.2 (OUT)
- net VCC: now also SW1.4 (B), SW2.4 (B), SW3.4 (B), SW4.4 (B)
- net more LEDS/data: now reaches D45.4 (DOUT)
- net at R5.2, SW4.1 (A), U4.13 (PD7): now also SW4.2 (A)
- net at R1.2, SW1.1 (A), U4.14 (PB0): now also SW1.2 (A)
- net at R3.2, SW2.1 (A), U4.5 (PD3): now also SW2.2 (A)
- net at C2.1, U1.1 (IN): now also J1.1 (POLE)
- net at R4.2, SW3.1 (A), U4.6 (PD4): now also SW3.2 (A)
- net MOSI: no longer names the net of U4.17 (PB3)
- net SCK: no longer names the net of U4.19 (PB5)
- net SS: no longer names the net of U4.16 (PB2)
- no-connect marks 26 -> 13
Other:
- added sheet more LEDS (untitled.kicad_sch)
- note removed: "MAX 7219 & LED Display"

Commit message: Update HPS_Round_Clock.kicad_sch
Parts:
- added C13, C14, C15, C16, C17, C18, C19, C20, C21, C22, C23, C24, C25, C26, C27, C28, C29, C30, C31, C32, C33, C34, C35, C36, C37, C38, C39, C40, C41, C42, C43, C44, C45, C46, C47, C48, C49, C50, C51, C52, C53, C54, C55, C56, C57, C58, C59, C60, C61, C62, C63, C64, C65, C66, C67, C68, C69, C70, C71, C72: C_0805_0.1uf, footprints:C_0805_2012Metric, symbol HPS:C_0805_0.1uf
- added H1, H2, H3, H4: MountingHole, footprints:MountingHole_3.2mm_M3, symbol HPS:MountingHole
Connections:
- net GND: now also C13.2, C14.2, C15.2, C16.2, C17.2, C18.2, C19.2, C20.2, C21.2, C22.2, C23.2, C24.2, C25.2, C26.2, C27.2, C28.2, C29.2, C30.2, C31.2, C32.2, C33.2, C34.2, C35.2, C36.2, C37.2, C38.2, C39.2, C40.2, C41.2, C42.2, C43.2, C44.2, C45.2, C46.2, C47.2, C48.2, C49.2, C50.2, C51.2, C52.2, C53.2, C54.2, C55.2, C56.2, C57.2, C58.2, C59.2, C60.2, C61.2, C62.2, C63.2, C64.2, C65.2, C66.2, C67.2, C68.2, C69.2, C70.2, C71.2, C72.2
- net VCC: now also C13.1, C14.1, C15.1, C16.1, C17.1, C18.1, C19.1, C20.1, C21.1, C22.1, C23.1, C24.1, C25.1, C26.1, C27.1, C28.1, C29.1, C30.1, C31.1, C32.1, C33.1, C34.1, C35.1, C36.1, C37.1, C38.1, C39.1, C40.1, C41.1, C42.1, C43.1, C44.1, C45.1, C46.1, C47.1, C48.1, C49.1, C50.1, C51.1, C52.1, C53.1, C54.1, C55.1, C56.1, C57.1, C58.1, C59.1, C60.1, C61.1, C62.1, C63.1, C64.1, C65.1, C66.1, C67.1, C68.1, C69.1, C70.1, C71.1, C72.1
Other:
- note added: "Capacitors (Connect one to each neopixel)"
