File: HPS_Round_Clock/HPS_Round_Clock.kicad_sch (KiCad schematic)
At the start: 144 parts, among them J1 Power_inlet_vertical, J2 Conn_01x06, SW1 Omron_B3F_SPST, SW2 Omron_B3F_SPST, SW3 Omron_B3F_SPST, SW4 Omron_B3F_SPST, SW5 Omron_B3F_SPST, U1 L7805, U2 DS1307_DIP-8, U4 ATmega328-PU, U5 TSOP38238, Y1 Crystal_16MHz, Y2 Crystal_32768Hz

Commit message: Update HPS_Round_Clock.kicad_sch
Parts:
- removed C10, C11, C12, C13, C14, C15, C16, C17, C18, C19, C20, C21, C22, C23, C24, C25, C26, C27, C28, C29, C30, C31, C32, C33, C34, C35, C36, C37, C8, C9: C_0805_0.1uf, footprints:C_0805_2012Metric, symbol HPS:C_0805_0.1uf

Commit message: Update HPS_Round_Clock.kicad_sch
Parts:
- added TP1, TP10, TP11, TP12, TP13, TP14, TP15, TP2, TP3, TP4, TP5, TP6, TP7, TP8, TP9: TestPoint, footprints:TestPoint_THTPad_D2.0mm_Drill1.0mm, symbol HPS:TestPoint
Connections:
- net GND: now also TP6.1
- net IR Receiver: now also TP3.1
- net Outer LED Ring: now also TP4.1
- net SCL: now also TP1.1
- net SDA: now also TP2.1
- net VCC: now also TP5.1
- net at U4.15 (PB1): now also TP7.1
- net at U4.16 (PB2): now also TP8.1
- net at U4.17 (PB3): now also TP9.1
- net at U4.18 (PB4): now also TP10.1
- net at U4.19 (PB5): now also TP11.1
- net at U4.23 (PC0): now also TP12.1
- net at U4.24 (PC1): now also TP13.1
- net at U4.25 (PC2): now also TP14.1
- net at U4.26 (PC3): now also TP15.1
- no-connect marks 13 -> 4
Other:
- moved on the sheet: R2

Commit message: Update HPS_Round_Clock.kicad_sch
Parts:
- removed TP10, TP9: TestPoint, footprints:TestPoint_THTPad_D2.0mm_Drill1.0mm, symbol HPS:TestPoint
- removed U5: TSOP38238, footprints:Vishay_MINICAST-3Pin, symbol HPS:TSOP38238
- added D66: LED_0805, footprints:LED_0805_2012Metric, symbol HPS:LED_0805
- added J3: Conn_02x03_Odd_Even, footprints:PinHeader_2x03_P2.54mm_Vertical, symbol HPS:Conn_02x03_Odd_Even
- added R10, R11: R_0805_4.7K, footprints:R_0805_2012Metric, symbol HPS:R_0805_4.7K
- added R8: R_0805_2.2K, footprints:R_0805_2012Metric, symbol HPS:R_0805_2.2K
- added U3: TSOP38238_Horiz, footprints:Vishay_MINICAST-3Pin_Horiz, symbol HPS:TSOP38238_Horiz
Connections:
- net GND: now also SW1.3 (B), SW1.4 (B), SW2.3 (B), SW2.4 (B), SW3.3 (B), SW3.4 (B), SW4.3 (B), SW4.4 (B), D66.1 (K), J3.6 (Pin_6), U3.2 (GND); no longer R1.1, R3.1, R4.1, R5.1
- net IR Receiver: now also U3.1 (OUT)
- net RESET: now also J3.5 (Pin_5)
- net SCL: now also R10.2
- net SDA: now also R11.2
- net VCC: now also R1.1, R3.2, R4.2, R5.2, J3.2 (Pin_2), R10.1, R11.1, U3.3 (Vs); no longer SW1.3 (B), SW1.4 (B), SW2.3 (B), SW2.4 (B), SW3.3 (B), SW3.4 (B), SW4.3 (B), SW4.4 (B)
- net at SW4.1 (A), SW4.2 (A), U4.13 (PD7): now also R5.1; no longer R5.2
- net MISO: now reaches U4.18 (MISO/PB4)
- net MISO: now also J3.1 (Pin_1)
- net at SW2.1 (A), SW2.2 (A), U4.5 (INT1/PD3): now also R3.1; no longer R3.2
- net at SW3.1 (A), SW3.2 (A), U4.6 (PD4): now also R4.1; no longer R4.2
- net MOSI: now reaches U4.17 (MOSI/PB3)
- net MOSI: now also J3.4 (Pin_4)
- new net: D66.2 (A), R8.2
- new net LED_SCK: J3.3 (Pin_3), R8.1
Other:
- note added: "Blinky LED"
- note added: "ICSP"
- note added: "Mounting Holes"
- moved on the sheet: H1, H2, H3, H4, R1, R3, R4, R5, SW2, SW4
