File: HPS_Round_Clock/HPS_Round_Clock.kicad_pcb (KiCad board)
At the start: 2 copper layers, 118 x 118 mm, 4 parts

Commit message: Update HPS_Round_Clock.kicad_pcb
Parts:
- added BT1: Battery_Cell, footprints:BatteryHolder_Keystone_106_1x20mm, F.Cu at (49.3, -2.54)
- added C1: C_0805_0.1uf, footprints:C_0805_2012Metric, F.Cu at (142.2, 71.1)
- added C11: C_0805_0.1uf, footprints:C_0805_2012Metric, F.Cu at (160.0, 137.2)
- added C12: C_0805_0.1uf, footprints:C_0805_2012Metric, F.Cu at (144.8, 66.0)
- added C13: C_0805_0.1uf, footprints:C_0805_2012Metric, F.Cu at (236.2, -40.6)
- added C14: C_0805_0.1uf, footprints:C_0805_2012Metric, F.Cu at (248.9, -40.6)
- added C15: C_0805_0.1uf, footprints:C_0805_2012Metric, F.Cu at (233.7, -48.3)
- added C16: C_0805_0.1uf, footprints:C_0805_2012Metric, F.Cu at (236.2, -30.5)
- added C2: C_0805_1uf, footprints:C_0805_2012Metric, F.Cu at (116.8, 86.4)
- added C3: C_0805_0.1uf, footprints:C_0805_2012Metric, F.Cu at (121.9, 30.5)
- added C4: C_0805_22pf, footprints:C_0805_2012Metric, F.Cu at (157.5, 71.1)
- added C5: C_0805_0.1uf, footprints:C_0805_2012Metric, F.Cu at (203.2, 53.3)
- added C6: C_0805_22pf, footprints:C_0805_2012Metric, F.Cu at (170.2, 86.4)
- added C61: C_0805_0.1uf, footprints:C_0805_2012Metric, F.Cu at (188.0, 91.4)
- added C62: C_0805_0.1uf, footprints:C_0805_2012Metric, F.Cu at (129.5, 121.9)
- added C63: C_0805_0.1uf, footprints:C_0805_2012Metric, F.Cu at (152.4, 66.0)
- added C7: C_0805_0.1uf, footprints:C_0805_2012Metric, F.Cu at (215.9, 144.8)
- added D1: NEOPIXEL_THT, footprints:Adafruit_Neopixel_TH_1938, F.Cu at (154.9, 58.4)
- added D10: NEOPIXEL_THT, footprints:Adafruit_Neopixel_TH_1938, F.Cu at (177.8, 78.7)
- added D11: NEOPIXEL_THT, footprints:Adafruit_Neopixel_TH_1938, F.Cu at (182.9, 83.8)
- added D12: NEOPIXEL_THT, footprints:Adafruit_Neopixel_TH_1938, F.Cu at (188.0, 83.8)
- added D13: NEOPIXEL_THT, footprints:Adafruit_Neopixel_TH_1938, F.Cu at (193.0, 88.9)
- added D14: NEOPIXEL_THT, footprints:Adafruit_Neopixel_TH_1938, F.Cu at (190.5, 96.5)
- added D15: NEOPIXEL_THT, footprints:Adafruit_Neopixel_TH_1938, F.Cu at (182.9, 99.1)
- added D16: NEOPIXEL_THT, footprints:Adafruit_Neopixel_TH_1938, F.Cu at (188.0, 104.1)
- added D17: NEOPIXEL_THT, footprints:Adafruit_Neopixel_TH_1938, F.Cu at (193.0, 109.2)
- added D18: NEOPIXEL_THT, footprints:Adafruit_Neopixel_TH_1938, F.Cu at (190.5, 116.8)
- added D19: NEOPIXEL_THT, footprints:Adafruit_Neopixel_TH_1938, F.Cu at (185.4, 119.4)
- added D2: NEOPIXEL_THT, footprints:Adafruit_Neopixel_TH_1938, F.Cu at (160.0, 55.9)
- added D20: NEOPIXEL_THT, footprints:Adafruit_Neopixel_TH_1938, F.Cu at (177.8, 119.4)
- added D21: NEOPIXEL_THT, footprints:Adafruit_Neopixel_TH_1938, F.Cu at (180.3, 127.0)
- added D22: NEOPIXEL_THT, footprints:Adafruit_Neopixel_TH_1938, F.Cu at (180.3, 134.6)
- added D23: NEOPIXEL_THT, footprints:Adafruit_Neopixel_TH_1938, F.Cu at (175.3, 137.2)
- added D24: NEOPIXEL_THT, footprints:Adafruit_Neopixel_TH_1938, F.Cu at (170.2, 137.2)
- added D25: NEOPIXEL_THT, footprints:Adafruit_Neopixel_TH_1938, F.Cu at (165.1, 132.1)
- added D26: NEOPIXEL_THT, footprints:Adafruit_Neopixel_TH_1938, F.Cu at (165.1, 139.7)
- added D27: NEOPIXEL_THT, footprints:Adafruit_Neopixel_TH_1938, F.Cu at (162.6, 144.8)
- added D28: NEOPIXEL_THT, footprints:Adafruit_Neopixel_TH_1938, F.Cu at (157.5, 147.3)
- added D29: NEOPIXEL_THT, footprints:Adafruit_Neopixel_TH_1938, F.Cu at (152.4, 142.2)
- added D3: NEOPIXEL_THT, footprints:Adafruit_Neopixel_TH_1938, F.Cu at (165.1, 55.9)
- added D30: NEOPIXEL_THT, footprints:Adafruit_Neopixel_TH_1938, F.Cu at (147.3, 137.2)
- added D31: NEOPIXEL_THT, footprints:Adafruit_Neopixel_TH_1938, F.Cu at (142.2, 142.2)
- added D32: NEOPIXEL_THT, footprints:Adafruit_Neopixel_TH_1938, F.Cu at (137.2, 144.8)
- added D33: NEOPIXEL_THT, footprints:Adafruit_Neopixel_TH_1938, F.Cu at (132.1, 142.2)
- added D34: NEOPIXEL_THT, footprints:Adafruit_Neopixel_TH_1938, F.Cu at (129.5, 137.2)
- added D35: NEOPIXEL_THT, footprints:Adafruit_Neopixel_TH_1938, F.Cu at (127.0, 132.1)
- added D36: NEOPIXEL_THT, footprints:Adafruit_Neopixel_TH_1938, F.Cu at (121.9, 134.6)
- added D37: NEOPIXEL_THT, footprints:Adafruit_Neopixel_TH_1938, F.Cu at (116.8, 134.6)
- added D38: NEOPIXEL_THT, footprints:Adafruit_Neopixel_TH_1938, F.Cu at (111.8, 129.5)
- added D39: NEOPIXEL_THT, footprints:Adafruit_Neopixel_TH_1938, F.Cu at (111.8, 121.9)
- added D4: NEOPIXEL_THT, footprints:Adafruit_Neopixel_TH_1938, F.Cu at (170.2, 61.0)
- added D40: NEOPIXEL_THT, footprints:Adafruit_Neopixel_TH_1938, F.Cu at (114.3, 116.8)
- added D41: NEOPIXEL_THT, footprints:Adafruit_Neopixel_TH_1938, F.Cu at (109.2, 116.8)
- added D42: NEOPIXEL_THT, footprints:Adafruit_Neopixel_TH_1938, F.Cu at (104.1, 114.3)
- added D43: NEOPIXEL_THT, footprints:Adafruit_Neopixel_TH_1938, F.Cu at (101.6, 106.7)
- added D44: NEOPIXEL_THT, footprints:Adafruit_Neopixel_TH_1938, F.Cu at (106.7, 101.6)
- added D45: NEOPIXEL_THT, footprints:Adafruit_Neopixel_TH_1938, F.Cu at (111.8, 99.1)
- added D46: NEOPIXEL_THT, footprints:Adafruit_Neopixel_TH_1938, F.Cu at (106.7, 96.5)
- added D47: NEOPIXEL_THT, footprints:Adafruit_Neopixel_TH_1938, F.Cu at (101.6, 91.4)
- added D48: NEOPIXEL_THT, footprints:Adafruit_Neopixel_TH_1938, F.Cu at (104.1, 83.8)
- added D49: NEOPIXEL_THT, footprints:Adafruit_Neopixel_TH_1938, F.Cu at (109.2, 81.3)
- added D5: NEOPIXEL_THT, footprints:Adafruit_Neopixel_TH_1938, F.Cu at (167.6, 68.6)
- added D50: NEOPIXEL_THT, footprints:Adafruit_Neopixel_TH_1938, F.Cu at (114.3, 81.3)
- added D51: NEOPIXEL_THT, footprints:Adafruit_Neopixel_TH_1938, F.Cu at (111.8, 76.2)
- added D52: NEOPIXEL_THT, footprints:Adafruit_Neopixel_TH_1938, F.Cu at (114.3, 68.6)
- added D53: NEOPIXEL_THT, footprints:Adafruit_Neopixel_TH_1938, F.Cu at (119.4, 63.5)
- added D54: NEOPIXEL_THT, footprints:Adafruit_Neopixel_TH_1938, F.Cu at (124.5, 63.5)
- added D55: NEOPIXEL_THT, footprints:Adafruit_Neopixel_TH_1938, F.Cu at (129.5, 68.6)
- added D56: NEOPIXEL_THT, footprints:Adafruit_Neopixel_TH_1938, F.Cu at (129.5, 61.0)
- added D57: NEOPIXEL_THT, footprints:Adafruit_Neopixel_TH_1938, F.Cu at (132.1, 55.9)
- added D58: NEOPIXEL_THT, footprints:Adafruit_Neopixel_TH_1938, F.Cu at (139.7, 53.3)
- added D59: NEOPIXEL_THT, footprints:Adafruit_Neopixel_TH_1938, F.Cu at (144.8, 58.4)
- added D6: NEOPIXEL_THT, footprints:Adafruit_Neopixel_TH_1938, F.Cu at (175.3, 66.0)
- added D60: NEOPIXEL_THT, footprints:Adafruit_Neopixel_TH_1938, F.Cu at (149.9, 61.0)
- added D61: NEOPIXEL_THT, footprints:Adafruit_Neopixel_TH_1938, F.Cu at (129.5, 33.0)
- added D62: NEOPIXEL_THT, footprints:Adafruit_Neopixel_TH_1938, F.Cu at (193.0, 40.6)
- added D63: NEOPIXEL_THT, footprints:Adafruit_Neopixel_TH_1938, F.Cu at (193.0, 50.8)
- added D64: NEOPIXEL_THT, footprints:Adafruit_Neopixel_TH_1938, F.Cu at (175.3, 162.6)
- added D65: NEOPIXEL_THT, footprints:Adafruit_Neopixel_TH_1938, F.Cu at (134.6, 180.3)
- added D66: NEOPIXEL_THT, footprints:Adafruit_Neopixel_TH_1938, F.Cu at (165.1, 170.2)
- added D67: NEOPIXEL_THT, footprints:Adafruit_Neopixel_TH_1938, F.Cu at (144.8, 167.6)
- added D68: NEOPIXEL_THT, footprints:Adafruit_Neopixel_TH_1938, F.Cu at (132.1, 170.2)
- added D69: NEOPIXEL_THT, footprints:Adafruit_Neopixel_TH_1938, F.Cu at (137.2, 162.6)
- added D7: NEOPIXEL_THT, footprints:Adafruit_Neopixel_TH_1938, F.Cu at (180.3, 66.0)
- added D70: NEOPIXEL_THT, footprints:Adafruit_Neopixel_TH_1938, F.Cu at (91.4, 68.6)
- added D71: NEOPIXEL_THT, footprints:Adafruit_Neopixel_TH_1938, F.Cu at (99.1, 61.0)
- added D72: NEOPIXEL_THT, footprints:Adafruit_Neopixel_TH_1938, F.Cu at (101.6, 27.9)
- added D73: LED_0805, footprints:LED_0805_2012Metric, F.Cu at (170.2, 94.0)
- added D8: NEOPIXEL_THT, footprints:Adafruit_Neopixel_TH_1938, F.Cu at (182.9, 71.1)
- added D9: NEOPIXEL_THT, footprints:Adafruit_Neopixel_TH_1938, F.Cu at (182.9, 76.2)
- added DS1: LED_Display_1001, footprints:Adafruit-1001-0-0-MFG, F.Cu at (147.3, 99.1)
- added J1: PJ-102AH, footprints:PJ-102AH, F.Cu at (124.5, 83.8)
- added J2: Conn_01x06, footprints:PinHeader_1x06_P2.54mm_Vertical, F.Cu at (119.4, 92.7)
- added R1: R_0805_10K, footprints:R_0805_2012Metric, F.Cu at (137.2, 68.6)
- added R2: R_0805_10K, footprints:R_0805_2012Metric, F.Cu at (205.7, 48.3)
- added R3: R_0805_10K, footprints:R_0805_2012Metric, F.Cu at (149.9, 71.1)
- added R4: R_0805_10K, footprints:R_0805_2012Metric, F.Cu at (167.6, 61.0)
- added R5: R_0805_10K, footprints:R_0805_2012Metric, F.Cu at (175.3, 114.3)
- added R6: R_0805_47, footprints:R_0805_2012Metric, F.Cu at (158.2, 63.5)
- added R7: R_0805_47, footprints:R_0805_2012Metric, F.Cu at (78.7, 114.3)
- added R8: R_0805_10K, footprints:R_0805_2012Metric, F.Cu at (142.2, 134.6)
- added R9: R_0805_1K, footprints:R_0805_2012Metric, F.Cu at (166.8, 100.3)
- added SW1: Omron_B3F_SPST, footprints:SW_SPST_Omron_B3FS-100xP, F.Cu at (127.0, 114.3)
- added SW2: Omron_B3F_SPST, footprints:SW_SPST_Omron_B3FS-100xP, F.Cu at (139.7, 114.3)
- added SW3: Omron_B3F_SPST, footprints:SW_SPST_Omron_B3FS-100xP, F.Cu at (154.9, 114.3)
- added SW4: Omron_B3F_SPST, footprints:SW_SPST_Omron_B3FS-100xP, F.Cu at (167.6, 114.3)
- added SW5: Omron_B3F_SPST, footprints:SW_SPST_Omron_B3FS-100xP, F.Cu at (203.2, 144.8)
- added U2: DS1307_DIP-8, footprints:DIP-8_W7.62mm, F.Cu at (174.0, 85.1)
- added U3: MAX7219, footprints:DIP-24_W7.62mm, F.Cu at (163.8, 120.7)
- added U4: ATmega328-PU, footprints:DIP-28_W7.62mm, F.Cu at (167.6, 76.2)
- added U5: TSOP38238, footprints:Vishay_MINICAST-3Pin, F.Cu at (161.2, 94.6)
- added Y1: Crystal_16MHz, footprints:Crystal_SMD_HC49-SD, F.Cu at (177.8, 104.1)
- added Y2: Crystal_32768Hz, footprints:Crystal_SMD_2Pin_3.2x1.5mm, F.Cu at (162.0, 100.6)
