File: HPS_Round_Clock/HPS_Round_Clock.kicad_pcb (KiCad board)
At the start: 2 copper layers, 118 x 118 mm, 117 parts, among them J1 PJ-102AH, J2 Conn_01x06, SW1 Omron_B3F_SPST, SW2 Omron_B3F_SPST, SW3 Omron_B3F_SPST, SW4 Omron_B3F_SPST, SW5 Omron_B3F_SPST, U2 DS1307_DIP-8, U3 MAX7219, U4 ATmega328-PU, U5 TSOP38238, Y1 Crystal_16MHz, Y2 Crystal_32768Hz

Commit message: Update HPS_Round_Clock.kicad_pcb
Parts:
- removed C14, C15, C16, C61, C62, C63: C_0805_0.1uf, footprints:C_0805_2012Metric
- removed D61, D62, D63, D64, D65, D66, D67, D68, D69, D70, D71, D72: NEOPIXEL_THT, footprints:Adafruit_Neopixel_TH_1938
- added C10: C_0805_0.1uf, footprints:C_0805_2012Metric, F.Cu at (111.8, 109.2)
- added C8: C_0805_0.1uf, footprints:C_0805_2012Metric, F.Cu at (181.6, 109.2)
- added C9: C_0805_0.1uf, footprints:C_0805_2012Metric, F.Cu at (109.2, 76.2)
- BT1: moved to B.Cu
- D1, D10, D11, D12, D13, D14, D15, D16, D17, D18, D19, D2, D20, D21, D22, D23, D24, D25, D26, D27, D28, D29, D3, D30, D31, D32, D33, D34, D35, D36, D37, D38, D39, D4, D40, D41, D42, D43, D44, D45, D46, D47, D48, D49, D5, D50, D51, D52, D53, D54, D55, D56, D57, D58, D59, D6, D60, D7, D8, D9: value NEOPIXEL_THT -> NEOPIXEL_SMT; footprint footprints:Adafruit_Neopixel_TH_1938 -> footprints:LED_SK6812_PLCC4_5.0x5.0mm_P3.2mm
- moved R7 155.8 mm to (210.8, 31.8)
- moved BT1 151.3 mm to (161.5, 99.1), turned to 180 degrees
- moved C13 126.7 mm to (149.9, 52.1)
- moved SW5 121.1 mm to (234.9, 27.9)
- moved J2 120.0 mm to (223.5, 33.0)
- moved C3 108.5 mm to (160.0, 132.1)
- moved C7 101.9 mm to (208.3, 43.2)
- moved R3 63.1 mm to (139.7, 133.3)
- moved C12 62.3 mm to (196.8, 100.3)
- moved R4 61.1 mm to (171.4, 121.9)
- moved R5 58.8 mm to (143.5, 64.8)
- moved Y1 55.9 mm to (127.0, 80.8)
- moved R6 55.7 mm to (207.0, 36.8)
- moved C4 53.0 mm to (119.4, 108.0)
- moved C6 51.8 mm to (125.7, 59.7)
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Connections:
- D60 pad 4: LEDs -> unconnected-(D60-Pad4)
- U4 pad 11: Inner LED Ring -> unconnected-(U4-Pad11)
Other:
- outline, holes or cut-outs redrawn

Commit message: Update HPS_Round_Clock.kicad_pcb
Parts:
- moved SW5 105.2 mm to (171.4, 111.8), turned to 180 degrees
- moved J2 84.3 mm to (180.3, 105.4), turned to 180 degrees
- moved BT1 79.8 mm to (209.7, 35.6)
- moved C9 79.6 mm to (175.3, 120.7), turned to -90 degrees
- moved C12 79.3 mm to (118.1, 91.0), turned to 90 degrees
- moved R7 74.4 mm to (176.5, 97.8), turned to 180 degrees
- moved C3 68.9 mm to (142.2, 65.5)
- moved R6 65.9 mm to (176.5, 95.2), turned to 180 degrees
- moved C7 58.8 mm to (176.5, 92.7), turned to 180 degrees
- moved R5 54.5 mm to (161.3, 116.3)
- moved C1 44.9 mm to (155.4, 66.0), turned to 180 degrees
- moved C10 42.0 mm to (144.8, 135.1), turned to -90 degrees
- moved R1 33.3 mm to (121.2, 106.7)
- moved R9 26.5 mm to (170.2, 77.5)
- moved D73 22.0 mm to (174.0, 77.5)
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Routing:
- net Net-(DS1-Pad1): track 0.00 -> 62.4 mm, vias 0 -> 1
- net Net-(DS1-Pad2): track 0.00 -> 55.0 mm, vias 0 -> 1
- net Net-(R5-Pad2): track 0.00 -> 53.5 mm, vias 0 -> 2
- net Net-(DS1-Pad3): track 0.00 -> 53.2 mm, vias 0 -> 1
- net Net-(R3-Pad2): track 0.00 -> 51.4 mm, vias 0 -> 2
- net SCK: track 0.00 -> 44.2 mm
- net Net-(DS1-Pad13): track 0.00 -> 40.9 mm
- net Net-(DS1-Pad4): track 0.00 -> 39.5 mm, vias 0 -> 1
- net Net-(C5-Pad1): track 0.00 -> 39.1 mm, vias 0 -> 2
- net Net-(DS1-Pad5): track 0.00 -> 37.2 mm
- net MOSI: track 0.00 -> 36.4 mm, vias 0 -> 1
- net GND: track 0.00 -> 36.3 mm
- net Net-(R1-Pad2): track 0.00 -> 35.9 mm, vias 0 -> 2
- net Net-(DS1-Pad12): track 0.00 -> 35.6 mm
- net Net-(DS1-Pad6): track 0.00 -> 34.0 mm
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Other:
- outline, holes or cut-outs redrawn

Commit message: Update HPS_Round_Clock.kicad_pcb
Parts:
- moved BT1 122.5 mm to (139.5, 135.9), turned to 0 degrees
- moved J1 49.9 mm to (171.4, 112.5), turned to 90 degrees
- moved C4 32.4 mm to (149.0, 71.1), turned to 0 degrees
- moved Y1 18.7 mm to (144.8, 74.9), turned to 0 degrees
- moved C6 18.2 mm to (141.0, 71.1), turned to 180 degrees
- moved U3 14.6 mm to (153.2, 109.0)
- moved C9 12.7 mm to (182.9, 110.5)
- moved R3 10.2 mm to (139.7, 126.5)
- moved R4 10.2 mm to (151.1, 126.5)
- moved R5 10.0 mm to (161.5, 126.4)
- moved SW1 9.87 mm to (126.8, 121.6)
- moved SW2 9.87 mm to (138.2, 121.6)
- moved SW3 9.87 mm to (149.0, 121.6)
- moved SW4 9.87 mm to (159.8, 121.6)
- moved SW5 9.87 mm to (171.3, 121.6)
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Routing:
- net Net-(DS1-Pad1): track 62.4 -> 0.00 mm, vias 1 -> 0
- net Net-(DS1-Pad2): track 55.0 -> 0.00 mm, vias 1 -> 0
- net Net-(R5-Pad2): track 53.5 -> 0.00 mm, vias 2 -> 0
- net Net-(DS1-Pad3): track 53.2 -> 0.00 mm, vias 1 -> 0
- net Net-(R3-Pad2): track 51.4 -> 0.00 mm, vias 2 -> 0
- net SCK: track 44.2 -> 0.00 mm
- net Net-(DS1-Pad13): track 40.9 -> 0.00 mm
- net Net-(DS1-Pad4): track 39.5 -> 0.00 mm, vias 1 -> 0
- net Net-(C5-Pad1): track 39.1 -> 0.00 mm, vias 2 -> 0
- net Net-(DS1-Pad5): track 37.2 -> 0.00 mm
- net MOSI: track 36.4 -> 0.00 mm, vias 1 -> 0
- net GND: track 36.3 -> 0.00 mm
- net Net-(R1-Pad2): track 35.9 -> 0.00 mm, vias 2 -> 0
- net Net-(DS1-Pad12): track 35.6 -> 0.00 mm
- net Net-(DS1-Pad6): track 34.0 -> 0.00 mm
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
Commit message: Update HPS_Round_Clock.kicad_pcb
Parts:
- removed D73: LED_0805, footprints:LED_0805_2012Metric
- removed DS1: LED_Display_1001, footprints:Adafruit-1001-0-0-MFG
- removed R8: R_0805_10K, footprints:R_0805_2012Metric
- removed U3: MAX7219, footprints:DIP-24_W7.62mm
- added C14: C_0805_0.1uf, footprints:C_0805_2012Metric, F.Cu at (144.2, 71.0)
- added D100: LED_0805, footprints:LED_0805_2012Metric, F.Cu at (149.0, 107.0)
- added D61: NEOPIXEL_SMT, footprints:LED_SK6812_PLCC4_5.0x5.0mm_P3.2mm, F.Cu at (126.5, 98.9)
- added D62: NEOPIXEL_SMT, footprints:LED_SK6812_PLCC4_5.0x5.0mm_P3.2mm, F.Cu at (127.6, 91.8)
- added D63: NEOPIXEL_SMT, footprints:LED_SK6812_PLCC4_5.0x5.0mm_P3.2mm, F.Cu at (130.9, 85.4)
- added D64: NEOPIXEL_SMT, footprints:LED_SK6812_PLCC4_5.0x5.0mm_P3.2mm, F.Cu at (135.9, 80.4)
- added D65: NEOPIXEL_SMT, footprints:LED_SK6812_PLCC4_5.0x5.0mm_P3.2mm, F.Cu at (142.3, 77.1)
- added U1: L7805, footprints:TO-252-2, F.Cu at (180.3, 115.6)
- J1: value PJ-102AH -> Power_inlet_vertical; footprint footprints:PJ-102AH -> footprints:Wurth-694106402002; moved to B.Cu
- moved D53 67.9 mm to (167.9, 112.3), turned to -36 degrees
- moved D52 67.7 mm to (171.1, 105.9), turned to -18 degrees
- moved C13 64.3 mm to (162.0, 123.0), turned to -54 degrees
- moved D57 64.3 mm to (142.3, 120.6), turned to -108 degrees
- moved C3 63.1 mm to (186.0, 111.0)
- moved D58 62.9 mm to (135.9, 117.4), turned to -126 degrees
- moved D54 62.2 mm to (162.8, 117.4), turned to -54 degrees
- moved D56 60.7 mm to (149.4, 121.7), turned to -90 degrees
- moved D51 59.9 mm to (172.2, 98.9), turned to 0 degrees
- moved C2 57.3 mm to (181.0, 109.0), turned to -39 degrees
- moved D48 57.0 mm to (162.8, 80.4), turned to 54 degrees
- moved D42 56.8 mm to (125.8, 61.3), turned to 122 degrees
- moved D55 55.9 mm to (156.4, 120.6), turned to -72 degrees
- moved D43 55.8 mm to (131.4, 58.3), turned to 114 degrees
- moved D49 54.9 mm to (167.9, 85.4), turned to 36 degrees
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Connections:
- net Net-(D45-Pad4) renamed /more LEDS/data
- D60 pad 4: unconnected-(D60-Pad4) -> Net-(D60-Pad4)
- SW1 pad 2: unconnected-(SW1-Pad2) -> Net-(R1-Pad2)
- SW1 pad 4: unconnected-(SW1-Pad4) -> VCC
- SW2 pad 2: unconnected-(SW2-Pad2) -> Net-(R3-Pad2)
- SW2 pad 4: unconnected-(SW2-Pad4) -> VCC
- SW3 pad 2: unconnected-(SW3-Pad2) -> Net-(R4-Pad2)
- SW3 pad 4: unconnected-(SW3-Pad4) -> VCC
- SW4 pad 2: unconnected-(SW4-Pad2) -> Net-(R5-Pad2)
- SW4 pad 4: unconnected-(SW4-Pad4) -> VCC
- U4 pad 16: SS -> unconnected-(U4-Pad16)
- U4 pad 17: MOSI -> unconnected-(U4-Pad17)
- U4 pad 19: SCK -> unconnected-(U4-Pad19)

Commit message: Update HPS_Round_Clock.kicad_pcb
Parts:
- moved D100 22.4 mm to (159.0, 87.0)
- moved R9 22.4 mm to (159.0, 89.4)
- moved U5 22.1 mm to (150.0, 87.0)
- moved C1 1.00 mm to (158.0, 94.0)
- moved C4 1.00 mm to (157.0, 112.0)
- moved C5 1.00 mm to (151.0, 94.0), turned to 180 degrees
- moved J2 0.65 mm to (153.0, 113.0)
Changed lines of the file:
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@@
   )
   (footprint "footprints:R_0805_2012Metric" (layer "F.Cu")
-    (at 149 109.381)
+    (at 159 89.381)
     (descr "Resistor SMD 0805 (2012 Metric), square (rectangular) end terminal, IPC_7351 nominal, (Body size source: http://www.tortai-tech.com/upload/download/2011102023233369053.pdf), generated with kicad-footprint-generator")
     (tags "resistor")
@@
     (property "Tolerance" "N/A")
     (attr smd)
-    (fp_text reference "R9" (at 1.27 -1.65) (layer "F.SilkS")
+    (fp_text reference "R9" (at 3 0.619) (layer "F.SilkS")
       (effects (font (size 1 1) (thickness 0.15)))
     )
@@
   )
   (footprint "footprints:C_0805_2012Metric" (layer "F.Cu")
-    (at 151 93 90)
+    (at 151 94 180)
     (descr "Capacitor SMD 0805 (2012 Metric), square (rectangular) end terminal, IPC_7351 nominal, (Body size source: http://www.tortai-tech.com/upload/download/2011102023233369053.pdf), generated with kicad-footprint-generator")
     (tags "capacitor")
@@
     (property "Voltage" "N/A")
     (attr smd)
-    (fp_text reference "C5" (at 0 -1.65 90) (layer "F.SilkS")
+    (fp_text reference "C5" (at -3 0) (layer "F.SilkS")
       (effects (font (size 1 1) (thickness 0.15)))
     )
-    (fp_text value "C_0805_0.1uf" (at 0 1.65 90) (layer "F.Fab")
+    (fp_text value "C_0805_0.1uf" (at 0 1.65) (layer "F.Fab")
       (effects (font (size 1 1) (thickness 0.15)))
     )
-    (fp_text user "${REFERENCE}" (at 0 0 90) (layer "F.Fab")
+    (fp_text user "${REFERENCE}" (at 0 0) (layer "F.Fab")
       (effects (font (size 0.5 0.5) (thickness 0.08)))
     )
@@
     (fp_line (start -1 0.6) (end -1 -0.6) (layer "F.Fab") (width 0.1))
     (fp_line (start 1 -0.6) (end 1 0.6) (layer "F.Fab") (width 0.1))
-    (pad "1" smd rect locked (at -0.85 0 90) (size 1.15 1.4) (layers "F.Cu" "F.Paste" "F.Mask")
+    (pad "1" smd rect locked (at -0.85 0 180) (size 1.15 1.4) (layers "F.Cu" "F.Paste" "F.Mask")
       (net 6 "Net-(C5-Pad1)") (pintype "passive"))
-    (pad "2" smd rect locked (at 0.85 0 90) (size 1.15 1.4) (layers "F.Cu" "F.Paste" "F.Mask")
+    (pad "2" smd rect locked (at 0.85 0 180) (size 1.15 1.4) (layers "F.Cu" "F.Paste" "F.Mask")
       (net 1 "GND") (pintype "passive"))
     (model "${HPS3DMOD}/C_0805_2012Metric.wrl"
@@
   )
   (footprint "footprints:LED_0805_2012Metric" (layer "F.Cu")
-    (at 149 107)
+    (at 159 87)
     (descr "LED SMD 0805 (2012 Metric), square (rectangular) end terminal, IPC_7351 nominal, (Body size source: https://docs.google.com/spreadsheets/d/1BsfQQcO9C6DZCsRaXUlFlo91Tg2WpOkGARC1WS5S8t0/edit?usp=sharing), generated with kicad-footprint-generator")
     (tags "LED")
@@
   )
   (footprint "footprints:C_0805_2012Metric" (layer "F.Cu")
-    (at 157 94 180)
+    (at 158 94 180)
     (descr "Capacitor SMD 0805 (2012 Metric), square (rectangular) end terminal, IPC_7351 nominal, (Body size source: http://www.tortai-tech.com/upload/download/2011102023233369053.pdf), generated with kicad-footprint-generator")
     (tags "capacitor")
@@
     (property "Voltage" "N/A")
     (attr smd)
-    (fp_text reference "C1" (at -2.032 2.54) (layer "F.SilkS")
+    (fp_text reference "C1" (at -3 0) (layer "F.SilkS")
       (effects (font (size 1 1) (thickness 0.15)))
     )
@@
   )
   (footprint "footprints:Vishay_MINICAST-3Pin" (layer "F.Cu")
-    (at 140.46 106.975)
+    (at 150 87)
     (descr "IR Receiver Vishay TSOP-xxxx, MINICAST package, see https://www.vishay.com/docs/82669/tsop32s40f.pdf")
     (tags "IR Receiver Vishay TSOP-xxxx MINICAST")
@@
     (property "Sheetname" "")
     (attr through_hole)
-    (fp_text reference "U5" (at 6.9977 4.835) (layer "F.SilkS")
+    (fp_text reference "U5" (at 2 -3) (layer "F.SilkS")
       (effects (font (size 1 1) (thickness 0.15)))
     )
@@
   )
   (footprint "footprints:PinHeader_1x06_P2.54mm_Vertical" (layer "F.Cu")
-    (at 152.35 113 -90)
+    (at 153 113 -90)
     (descr "Through hole straight pin header, 1x06, 2.54mm pitch, single row")
     (tags "Through hole pin header THT 1x06 2.54mm single row")
@@
   )
   (footprint "footprints:C_0805_2012Metric" (layer "F.Cu")
-    (at 156 112 180)
+    (at 157 112 180)
     (descr "Capacitor SMD 0805 (2012 Metric), square (rectangular) end terminal, IPC_7351 nominal, (Body size source: http://www.tortai-tech.com/upload/download/2011102023233369053.pdf), generated with kicad-footprint-generator")
     (tags "capacitor")

Commit message: Update HPS_Round_Clock.kicad_pcb
Parts:
- added C15: C_0805_0.1uf, footprints:C_0805_2012Metric, F.Cu at (197.5, 120.0)
- added C16: C_0805_0.1uf, footprints:C_0805_2012Metric, F.Cu at (190.0, 132.5)
- added C17: C_0805_0.1uf, footprints:C_0805_2012Metric, F.Cu at (105.0, 125.0)
- added C18: C_0805_0.1uf, footprints:C_0805_2012Metric, F.Cu at (112.5, 99.0)
- added C19: C_0805_0.1uf, footprints:C_0805_2012Metric, F.Cu at (150.0, 62.6)
- added C20: C_0805_0.1uf, footprints:C_0805_2012Metric, F.Cu at (130.4, 122.1)
- added C21: C_0805_0.1uf, footprints:C_0805_2012Metric, F.Cu at (160.0, 64.0)
- added C22: C_0805_0.1uf, footprints:C_0805_2012Metric, F.Cu at (115.0, 137.5)
- added C23: C_0805_0.1uf, footprints:C_0805_2012Metric, F.Cu at (155.0, 63.0)
- added C24: C_0805_0.1uf, footprints:C_0805_2012Metric, F.Cu at (125.0, 117.5)
- added C25: C_0805_0.1uf, footprints:C_0805_2012Metric, F.Cu at (200.0, 112.5)
- added C26: C_0805_0.1uf, footprints:C_0805_2012Metric, F.Cu at (120.5, 107.5)
- added C27: C_0805_0.1uf, footprints:C_0805_2012Metric, F.Cu at (169.1, 118.5)
- added C28: C_0805_0.1uf, footprints:C_0805_2012Metric, F.Cu at (186.7, 87.6)
- added C29: C_0805_0.1uf, footprints:C_0805_2012Metric, F.Cu at (170.0, 69.0)
- added C30: C_0805_0.1uf, footprints:C_0805_2012Metric, F.Cu at (137.5, 150.0)
- added C31: C_0805_0.1uf, footprints:C_0805_2012Metric, F.Cu at (100.0, 112.5)
- added C32: C_0805_0.1uf, footprints:C_0805_2012Metric, F.Cu at (188.0, 97.8)
- added C33: C_0805_0.1uf, footprints:C_0805_2012Metric, F.Cu at (130.3, 68.5)
- added C34: C_0805_0.1uf, footprints:C_0805_2012Metric, F.Cu at (140.0, 64.0)
- added C35: C_0805_0.1uf, footprints:C_0805_2012Metric, F.Cu at (142.5, 151.1)
- added C36: C_0805_0.1uf, footprints:C_0805_2012Metric, F.Cu at (125.0, 145.0)
- added C37: C_0805_0.1uf, footprints:C_0805_2012Metric, F.Cu at (140.0, 70.0)
- added C38: C_0805_0.1uf, footprints:C_0805_2012Metric, F.Cu at (162.5, 150.0)
- added C39: C_0805_0.1uf, footprints:C_0805_2012Metric, F.Cu at (110.0, 132.5)
- added C40: C_0805_0.1uf, footprints:C_0805_2012Metric, F.Cu at (122.0, 75.0)
- added C41: C_0805_0.1uf, footprints:C_0805_2012Metric, F.Cu at (153.7, 125.4)
- added C42: C_0805_0.1uf, footprints:C_0805_2012Metric, F.Cu at (185.0, 137.5)
- added C43: C_0805_0.1uf, footprints:C_0805_2012Metric, F.Cu at (186.0, 104.0)
- added C44: C_0805_0.1uf, footprints:C_0805_2012Metric, F.Cu at (120.0, 90.0)
- added C45: C_0805_0.1uf, footprints:C_0805_2012Metric, F.Cu at (180.0, 99.0)
- added C46: C_0805_0.1uf, footprints:C_0805_2012Metric, F.Cu at (102.5, 120.0)
- added C47: C_0805_0.1uf, footprints:C_0805_2012Metric, F.Cu at (114.0, 89.0)
- added C48: C_0805_0.1uf, footprints:C_0805_2012Metric, F.Cu at (177.4, 74.6)
- added C49: C_0805_0.1uf, footprints:C_0805_2012Metric, F.Cu at (180.0, 142.5)
- added C50: C_0805_0.1uf, footprints:C_0805_2012Metric, F.Cu at (120.0, 142.5)
- added C51: C_0805_0.1uf, footprints:C_0805_2012Metric, F.Cu at (144.5, 126.3)
- added C52: C_0805_0.1uf, footprints:C_0805_2012Metric, F.Cu at (180.0, 90.0)
- added C53: C_0805_0.1uf, footprints:C_0805_2012Metric, F.Cu at (135.0, 66.0)
- added C54: C_0805_0.1uf, footprints:C_0805_2012Metric, F.Cu at (167.5, 72.5)
- added C55: C_0805_0.1uf, footprints:C_0805_2012Metric, F.Cu at (113.0, 94.0)
- added C56: C_0805_0.1uf, footprints:C_0805_2012Metric, F.Cu at (119.0, 79.0)
- added C57: C_0805_0.1uf, footprints:C_0805_2012Metric, F.Cu at (158.8, 68.8)
- added C58: C_0805_0.1uf, footprints:C_0805_2012Metric, F.Cu at (116.0, 84.0)
- added C59: C_0805_0.1uf, footprints:C_0805_2012Metric, F.Cu at (113.0, 104.0)
- added C60: C_0805_0.1uf, footprints:C_0805_2012Metric, F.Cu at (195.0, 125.0)
- added C61: C_0805_0.1uf, footprints:C_0805_2012Metric, F.Cu at (130.8, 74.5)
- added C62: C_0805_0.1uf, footprints:C_0805_2012Metric, F.Cu at (124.2, 80.7)
- added C63: C_0805_0.1uf, footprints:C_0805_2012Metric, F.Cu at (174.3, 146.1)
- added C64: C_0805_0.1uf, footprints:C_0805_2012Metric, F.Cu at (157.5, 150.8)
- added C65: C_0805_0.1uf, footprints:C_0805_2012Metric, F.Cu at (175.0, 80.0)
- added C66: C_0805_0.1uf, footprints:C_0805_2012Metric, F.Cu at (173.7, 71.5)
- added C67: C_0805_0.1uf, footprints:C_0805_2012Metric, F.Cu at (132.5, 148.3)
- added C68: C_0805_0.1uf, footprints:C_0805_2012Metric, F.Cu at (179.2, 105.0)
- added C69: C_0805_0.1uf, footprints:C_0805_2012Metric, F.Cu at (188.0, 92.7)
- added C70: C_0805_0.1uf, footprints:C_0805_2012Metric, F.Cu at (165.0, 66.0)
- added C71: C_0805_0.1uf, footprints:C_0805_2012Metric, F.Cu at (182.9, 78.7)
- added C72: C_0805_0.1uf, footprints:C_0805_2012Metric, F.Cu at (117.5, 100.0)
- moved C9 15.3 mm to (167.6, 148.6), turned to -160 degrees
- moved R2 13.9 mm to (169.0, 133.6), turned to 132 degrees
- moved C14 6.82 mm to (150.0, 67.5)
- moved C8 5.33 mm to (185.4, 82.5), turned to -64 degrees
- moved C11 3.16 mm to (126.3, 71.5), turned to 38 degrees
- moved C12 2.24 mm to (145.0, 63.0), turned to -172 degrees
- turned D100 to 180 degrees
Routing:
- net VCC: track 0.00 -> 116.4 mm
- net GND: track 0.00 -> 99.7 mm
- net Net-(R1-Pad2): track 0.00 -> 72.3 mm, vias 0 -> 1
- net Net-(BT1-Pad1): track 0.00 -> 45.8 mm, vias 0 -> 1
- net Net-(R3-Pad2): track 0.00 -> 39.8 mm, vias 0 -> 1
- net IR Receiver: track 0.00 -> 30.2 mm, vias 0 -> 1
- net Net-(C6-Pad2): track 0.00 -> 13.0 mm
- net Net-(R5-Pad2): track 0.00 -> 11.1 mm
- net RESET: track 0.00 -> 11.0 mm
- net Net-(R4-Pad2): track 0.00 -> 10.5 mm
- net Net-(C4-Pad2): track 0.00 -> 9.10 mm
- net SCL: track 0.00 -> 9.00 mm
- net Net-(D57-Pad4): track 0.00 -> 8.17 mm
- net Net-(D47-Pad4): track 0.00 -> 8.06 mm
- net Net-(D52-Pad4): track 0.00 -> 7.82 mm
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
Commit message: Update HPS_Round_Clock.kicad_pcb
Parts:
- removed C10, C11, C12, C13, C14, C15, C16, C17, C18, C19, C20, C21, C22, C23, C24, C25, C26, C27, C28, C29, C30, C31, C32, C33, C34, C35, C36, C37, C8, C9: C_0805_0.1uf, footprints:C_0805_2012Metric
- moved C62 33.6 mm to (112.9, 112.3)
- moved C40 23.7 mm to (141.6, 61.6), turned to -87 degrees
- moved C56 19.6 mm to (132.5, 64.8), turned to -64 degrees
- moved C53 19.4 mm to (153.6, 60.5), turned to -96 degrees
- moved C48 15.4 mm to (187.3, 86.4), turned to -158 degrees
- moved C58 14.8 mm to (123.2, 71.1), turned to -56 degrees
- moved C42 14.6 mm to (182.2, 123.2), turned to 134 degrees
- moved C63 13.4 mm to (164.7, 136.7), turned to 108 degrees
- moved C49 13.1 mm to (174.0, 130.8), turned to 126 degrees
- moved C60 11.5 mm to (185.5, 118.5), turned to 150 degrees
- moved C47 9.87 mm to (116.2, 79.4), turned to -33 degrees
- moved C55 5.16 mm to (112.2, 88.9), turned to -20 degrees
- moved C43 5.10 mm to (189.2, 108.0), turned to 169 degrees
- moved C69 4.76 mm to (189.7, 97.2), turned to 180 degrees
- moved R5 4.64 mm to (154.9, 138.4)
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Routing:
- net VCC: track 116.4 -> 0.00 mm
- net Outer LED Ring: track 0.00 -> 65.4 mm, vias 0 -> 3
- net RESET: track 11.0 -> 72.9 mm, vias 0 -> 3
- net GND: track 99.7 -> 140.9 mm, vias 0 -> 60
- net Net-(R5-Pad2): track 11.1 -> 44.4 mm, vias 0 -> 2
- net Net-(R4-Pad2): track 10.5 -> 39.9 mm, vias 0 -> 2
- net /more LEDS/data: track 0.00 -> 18.8 mm, vias 0 -> 2
- net Net-(C2-Pad1): track 0.00 -> 14.5 mm, vias 0 -> 1
- net Net-(J2-Pad4): track 0.00 -> 9.83 mm, vias 0 -> 1
- net Net-(C7-Pad1): track 0.00 -> 8.41 mm
- net Net-(J2-Pad5): track 0.00 -> 7.67 mm
- net IR Receiver: track 30.2 -> 35.1 mm, vias 1 -> 3
- net Net-(R1-Pad2): track 72.3 -> 67.8 mm, vias 1 -> 3
- net TXD: track 0.00 -> 3.70 mm
- net RXD: track 0.00 -> 3.70 mm
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- added copper zone on B.Cu, net GND
- added copper zone on F.Cu, net VCC

Commit message: Update HPS_Round_Clock.kicad_pcb
Parts:
- moved C64 38.4 mm to (132.1, 121.9), turned to -127 degrees
- moved C41 36.1 mm to (178.4, 99.1), turned to 3 degrees
- moved C45 26.7 mm to (166.3, 121.9), turned to -45 degrees
- moved C38 18.2 mm to (144.5, 152.6), turned to -108 degrees
- moved C42 15.3 mm to (186.7, 137.8), turned to -46 degrees
- moved C49 15.3 mm to (175.3, 146.1), turned to -54 degrees
- moved C63 15.0 mm to (160.7, 151.1), turned to -72 degrees
- moved C60 12.2 mm to (195.0, 126.2), turned to -30 degrees
- moved C72 10.2 mm to (121.9, 109.2), turned to 180 degrees
- moved C57 9.61 mm to (149.2, 69.8), turned to 90 degrees
- moved C62 6.40 mm to (111.8, 106.0), turned to 9 degrees
- moved R5 5.16 mm to (160.0, 139.3), turned to 18 degrees
- moved C1 3.75 mm to (154.3, 93.3), turned to 0 degrees
- moved C52 3.47 mm to (176.5, 90.0), turned to 18 degrees
- moved C54 3.27 mm to (166.4, 75.6), turned to 54 degrees
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Routing:
- net GND: track 140.9 -> 258.0 mm, vias 60 -> 113
- net Net-(C2-Pad1): track 14.5 -> 18.3 mm
- net Net-(R5-Pad2): track 44.4 -> 47.8 mm
- net Net-(D60-Pad4): track 6.72 -> 8.85 mm
- net Net-(D57-Pad4): track 8.17 -> 6.79 mm
- net Net-(D54-Pad4): track 7.70 -> 6.69 mm
- net Net-(C7-Pad1): track 8.41 -> 7.40 mm
- net Net-(R1-Pad2): track 67.8 -> 68.5 mm
- net Net-(J2-Pad4): track 9.83 -> 9.20 mm
