File: HPS_Round_Clock/HPS_Round_Clock.kicad_pcb (KiCad board)
At the start: 2 copper layers, 118 x 118 mm, 134 parts, among them J1 Power_inlet_vertical, J2 Conn_01x06, SW1 Omron_B3F_SPST, SW2 Omron_B3F_SPST, SW3 Omron_B3F_SPST, SW4 Omron_B3F_SPST, SW5 Omron_B3F_SPST, U1 L7805, U2 DS1307_DIP-8, U4 ATmega328-PU, U5 TSOP38238, Y1 Crystal_16MHz, Y2 Crystal_32768Hz

Commit message: Update HPS_Round_Clock.kicad_pcb
Parts:
- added TP1: TestPoint, footprints:TestPoint_THTPad_D2.0mm_Drill1.0mm, F.Cu at (133.3, 93.3)
- added TP10: TestPoint, footprints:TestPoint_THTPad_D2.0mm_Drill1.0mm, F.Cu at (157.5, 99.7)
- added TP11: TestPoint, footprints:TestPoint_THTPad_D2.0mm_Drill1.0mm, F.Cu at (155.6, 93.3)
- added TP12: TestPoint, footprints:TestPoint_THTPad_D2.0mm_Drill1.0mm, F.Cu at (148.0, 99.7)
- added TP13: TestPoint, footprints:TestPoint_THTPad_D2.0mm_Drill1.0mm, F.Cu at (142.9, 99.7)
- added TP14: TestPoint, footprints:TestPoint_THTPad_D2.0mm_Drill1.0mm, F.Cu at (138.4, 99.7)
- added TP15: TestPoint, footprints:TestPoint_THTPad_D2.0mm_Drill1.0mm, F.Cu at (135.3, 99.7)
- added TP2: TestPoint, footprints:TestPoint_THTPad_D2.0mm_Drill1.0mm, F.Cu at (134.6, 89.5)
- added TP3: TestPoint, footprints:TestPoint_THTPad_D2.0mm_Drill1.0mm, F.Cu at (144.1, 108.0)
- added TP4: TestPoint, footprints:TestPoint_THTPad_D2.0mm_Drill1.0mm, F.Cu at (148.0, 61.6)
- added TP5: TestPoint, footprints:TestPoint_THTPad_D2.0mm_Drill1.0mm, F.Cu at (183.5, 94.6)
- added TP6: TestPoint, footprints:TestPoint_THTPad_D2.0mm_Drill1.0mm, F.Cu at (116.8, 95.2)
- added TP7: TestPoint, footprints:TestPoint_THTPad_D2.0mm_Drill1.0mm, F.Cu at (165.7, 93.3)
- added TP8: TestPoint, footprints:TestPoint_THTPad_D2.0mm_Drill1.0mm, F.Cu at (163.8, 99.7)
- added TP9: TestPoint, footprints:TestPoint_THTPad_D2.0mm_Drill1.0mm, F.Cu at (160.0, 93.3)
- moved C1 1.58 mm to (152.8, 92.9), turned to 90 degrees
- moved D100 1.04 mm to (158.9, 86.0)
- moved R9 1.04 mm to (158.9, 88.4)
- moved U5 1.04 mm to (149.9, 86.0)
Connections:
- U4 pad 15: unconnected-(U4-Pad15) -> Net-(TP7-Pad1)
- U4 pad 16: unconnected-(U4-Pad16) -> Net-(TP8-Pad1)
- U4 pad 17: unconnected-(U4-Pad17) -> Net-(TP9-Pad1)
- U4 pad 18: unconnected-(U4-Pad18) -> Net-(TP10-Pad1)
- U4 pad 19: unconnected-(U4-Pad19) -> Net-(TP11-Pad1)
- U4 pad 23: unconnected-(U4-Pad23) -> Net-(TP12-Pad1)
- U4 pad 24: unconnected-(U4-Pad24) -> Net-(TP13-Pad1)
- U4 pad 25: unconnected-(U4-Pad25) -> Net-(TP14-Pad1)
- U4 pad 26: unconnected-(U4-Pad26) -> Net-(TP15-Pad1)
Routing:
- net SDA: track 3.92 -> 12.1 mm, vias 0 -> 1
- net Net-(TP15-Pad1): track 0.00 -> 4.28 mm
- net Net-(TP14-Pad1): track 0.00 -> 4.02 mm
- net Net-(TP10-Pad1): track 0.00 -> 3.49 mm
- net Net-(TP9-Pad1): track 0.00 -> 3.49 mm
- net Net-(TP8-Pad1): track 0.00 -> 3.39 mm
- net SCL: track 9.00 -> 12.4 mm
- net Net-(TP11-Pad1): track 0.00 -> 3.23 mm
- net Net-(TP13-Pad1): track 0.00 -> 3.23 mm
- net Net-(TP7-Pad1): track 0.00 -> 3.23 mm
- net IR Receiver: track 35.0 -> 37.7 mm
- net Outer LED Ring: track 65.4 -> 68.1 mm
- net Net-(D100-Pad1): track 2.42 -> 0.00 mm
- net Net-(J2-Pad4): track 9.20 -> 7.16 mm
- net GND: track 258.0 -> 258.8 mm

Commit message: Update HPS_Round_Clock.kicad_pcb
Parts:
- moved TP14 16.7 mm to (141.0, 83.2), turned to -90 degrees
- moved C1 15.4 mm to (149.2, 108.0), turned to -90 degrees
- moved TP13 11.4 mm to (149.2, 90.2), turned to -90 degrees
- moved TP10 9.61 mm to (158.8, 90.2)
- moved TP8 9.55 mm to (164.5, 90.2)
- moved TP12 6.48 mm to (149.2, 93.3), turned to -90 degrees
- moved TP15 5.97 mm to (135.0, 93.7), turned to -90 degrees
- moved C5 3.50 mm to (152.8, 92.1), turned to 90 degrees
- moved TP6 3.24 mm to (113.7, 94.6)
- moved U5 2.78 mm to (149.9, 83.2)
- moved TP1 2.16 mm to (133.2, 91.2)
- moved D100 1.69 mm to (158.1, 84.5)
- moved R9 1.69 mm to (158.1, 86.8)
- moved TP2 1.33 mm to (135.0, 88.3)
- moved TP11 0.76 mm to (155.6, 92.6)
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Routing:
- net SCL: track 12.4 -> 23.5 mm, vias 0 -> 1
- net Net-(TP13-Pad1): track 3.23 -> 13.7 mm, vias 0 -> 1
- net Net-(TP14-Pad1): track 4.02 -> 14.2 mm
- net SDA: track 12.1 -> 20.0 mm, vias 1 -> 2
- net IR Receiver: track 37.7 -> 43.3 mm
- net Net-(TP12-Pad1): track 0.00 -> 5.00 mm
- net Net-(TP10-Pad1): track 3.49 -> 7.94 mm
- net Net-(TP8-Pad1): track 3.39 -> 6.82 mm
- net Net-(D100-Pad1): track 0.00 -> 2.42 mm
- net Net-(BT1-Pad1): track 44.5 -> 42.2 mm
- net Net-(R1-Pad2): track 68.1 -> 70.3 mm
- net Net-(D60-Pad4): track 8.85 -> 6.83 mm
- net Net-(C5-Pad1): track 2.56 -> 4.49 mm
- net GND: track 258.8 -> 257.4 mm
- net RESET: track 73.1 -> 73.9 mm
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
Commit message: Update HPS_Round_Clock.kicad_pcb
Parts:
- moved TP11 25.9 mm to (154.9, 66.7)
- moved TP9 25.0 mm to (163.2, 68.6)
- moved TP15 23.6 mm to (130.8, 70.5)
- moved TP10 22.9 mm to (158.8, 67.3)
- moved TP2 20.4 mm to (137.2, 67.9)
- moved TP7 20.3 mm to (171.4, 73.7)
- moved TP8 19.9 mm to (167.6, 70.5)
- moved TP1 16.8 mm to (125.7, 76.2)
- moved TP14 16.7 mm to (143.5, 66.7)
- moved C3 13.5 mm to (172.7, 116.2)
- moved TP4 4.84 mm to (149.9, 66.0)
- moved C70 0.90 mm to (165.1, 63.5), turned to -99 degrees
Routing:
- net Net-(TP11-Pad1): track 3.23 -> 30.8 mm
- net Net-(TP9-Pad1): track 3.49 -> 29.8 mm, vias 0 -> 1
- net Net-(TP15-Pad1): track 4.02 -> 29.1 mm, vias 0 -> 1
- net SCL: track 23.5 -> 47.6 mm, vias 1 -> 3
- net Net-(TP8-Pad1): track 6.82 -> 29.8 mm, vias 0 -> 1
- net Net-(TP7-Pad1): track 3.39 -> 25.2 mm
- net Net-(TP10-Pad1): track 7.94 -> 29.5 mm
- net SDA: track 20.0 -> 40.8 mm, vias 2 -> 3
- net Net-(TP14-Pad1): track 14.2 -> 32.2 mm, vias 0 -> 1
- net Net-(BT1-Pad1): track 42.2 -> 46.2 mm
- net GND: track 257.4 -> 258.4 mm
- net Net-(C2-Pad1): track 18.3 -> 19.2 mm
- net Outer LED Ring: track 68.1 -> 67.3 mm

Commit message: Update HPS_Round_Clock.kicad_pcb
Parts:
- J2: moved to B.Cu
- turned J2 to 90 degrees
Changed lines of the file:
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@@
-    )
-  )
-  (footprint "footprints:PinHeader_1x06_P2.54mm_Vertical" (layer "F.Cu")
-    (at 153 113 -90)
-    (descr "Through hole straight pin header, 1x06, 2.54mm pitch, single row")
-    (tags "Through hole pin header THT 1x06 2.54mm single row")
-    (property "Digikey PN" "732-5319-ND")
-    (property "MFG" "Würth Elektronik")
-    (property "MPN" "61300611121")
-    (property "Mouser PN" "N/A")
-    (property "Sheetfile" "HPS_Round_Clock.kicad_sch")
-    (property "Sheetname" "")
-    (attr smd)
-    (fp_text reference "J2" (at 3 2.35 90) (layer "F.SilkS")
-      (effects (font (size 1 1) (thickness 0.15)))
-    )
-    (fp_text value "Conn_01x06" (at 0 15.03 90) (layer "F.Fab")
-      (effects (font (size 1 1) (thickness 0.15)))
-    )
-    (fp_text user "${REFERENCE}" (at 0 6.35) (layer "F.Fab")
-      (effects (font (size 1 1) (thickness 0.15)))
-    )
-    (fp_line (start 1.33 1.27) (end 1.33 14.03) (layer "F.SilkS") (width 0.12))
-    (fp_line (start -1.33 1.27) (end 1.33 1.27) (layer "F.SilkS") (width 0.12))
-    (fp_line (start -1.33 -1.33) (end 0 -1.33) (layer "F.SilkS") (width 0.12))
-    (fp_line (start -1.33 0) (end -1.33 -1.33) (layer "F.SilkS") (width 0.12))
-    (fp_line (start -1.33 1.27) (end -1.33 14.03) (layer "F.SilkS") (width 0.12))
-    (fp_line (start -1.33 14.03) (end 1.33 14.03) (layer "F.SilkS") (width 0.12))
-    (fp_line (start 1.8 -1.8) (end -1.8 -1.8) (layer "F.CrtYd") (width 0.05))
-    (fp_line (start -1.8 14.5) (end 1.8 14.5) (layer "F.CrtYd") (width 0.05))
-    (fp_line (start 1.8 14.5) (end 1.8 -1.8) (layer "F.CrtYd") (width 0.05))
-    (fp_line (start -1.8 -1.8) (end -1.8 14.5) (layer "F.CrtYd") (width 0.05))
-    (fp_line (start 1.27 13.97) (end -1.27 13.97) (layer "F.Fab") (width 0.1))
-    (fp_line (start 1.27 -1.27) (end 1.27 13.97) (layer "F.Fab") (width 0.1))
-    (fp_line (start -0.635 -1.27) (end 1.27 -1.27) (layer "F.Fab") (width 0.1))
-    (fp_line (start -1.27 13.97) (end -1.27 -0.635) (layer "F.Fab") (width 0.1))
-    (fp_line (start -1.27 -0.635) (end -0.635 -1.27) (layer "F.Fab") (width 0.1))
-    (pad "1" thru_hole rect locked (at 0 0 270) (size 1.7 1.7) (drill 1) (layers *.Cu *.Mask)
-      (net 1 "GND") (pinfunction "Pin_1") (pintype "passive"))
-    (pad "2" thru_hole oval locked (at 0 2.54 270) (size 1.7 1.7) (drill 1) (layers *.Cu *.Mask)
-      (net 1 "GND") (pinfunction "Pin_2") (pintype "passive"))
-    (pad "3" thru_hole oval locked (at 0 5.08 270) (size 1.7 1.7) (drill 1) (layers *.Cu *.Mask)
-      (net 62 "unconnected-(J2-Pad3)") (pinfunction "Pin_3") (pintype "passive+no_connect"))
-    (pad "4" thru_hole oval locked (at 0 7.62 270) (size 1.7 1.7) (drill 1) (layers *.Cu *.Mask)
-      (net 61 "Net-(J2-Pad4)") (pinfunction "Pin_4") (pintype "passive"))
-    (pad "5" thru_hole oval locked (at 0 10.16 270) (size 1.7 1.7) (drill 1) (layers *.Cu *.Mask)
-      (net 60 "Net-(J2-Pad5)") (pinfunction "Pin_5") (pintype "passive"))
-    (pad "6" thru_hole oval locked (at 0 12.7 270) (size 1.7 1.7) (drill 1) (layers *.Cu *.Mask)
-      (net 8 "Net-(C7-Pad1)") (pinfunction "Pin_6") (pintype "passive"))
-    (model "${HPS3DMOD}/PinHeader_1x06_P2.54mm_Vertical.wrl"
-      (offset (xyz 0 0 0))
-      (scale (xyz 1 1 1))
-      (rotate (xyz 0 0 0))
     )
   )
@@
       (offset (xyz 0 0 0))
       (scale (xyz 1 1 1))
+      (rotate (xyz 0 0 0))
+    )
+  )
+  (footprint "footprints:PinHeader_1x06_P2.54mm_Vertical" (layer "B.Cu")
+    (at 153.035 113.03 90)
+    (descr "Through hole straight pin header, 1x06, 2.54mm pitch, single row")
+    (tags "Through hole pin header THT 1x06 2.54mm single row")
+    (property "Digikey PN" "732-5319-ND")
+    (property "MFG" "Würth Elektronik")
+    (property "MPN" "61300611121")
+    (property "Mouser PN" "N/A")
+    (property "Sheetfile" "HPS_Round_Clock.kicad_sch")
+    (property "Sheetname" "")
+    (attr smd)
+    (fp_text reference "J2" (at 3 -2.35 90) (layer "B.SilkS")
+      (effects (font (size 1 1) (thickness 0.15)) (justify mirror))
+    )
+    (fp_text value "Conn_01x06" (at 0 -15.03 90) (layer "B.Fab")
+      (effects (font (size 1 1) (thickness 0.15)) (justify mirror))
+    )
+    (fp_text user "${REFERENCE}" (at 0 -6.35) (layer "B.Fab")
+      (effects (font (size 1 1) (thickness 0.15)) (justify mirror))
+    )
+    (fp_line (start 1.33 -1.27) (end 1.33 -14.03) (layer "B.SilkS") (width 0.12))
+    (fp_line (start -1.33 -1.27) (end 1.33 -1.27) (layer "B.SilkS") (width 0.12))
+    (fp_line (start -1.33 1.33) (end 0 1.33) (layer "B.SilkS") (width 0.12))
+    (fp_line (start -1.33 0) (end -1.33 1.33) (layer "B.SilkS") (width 0.12))
+    (fp_line (start -1.33 -1.27) (end -1.33 -14.03) (layer "B.SilkS") (width 0.12))
+    (fp_line (start -1.33 -14.03) (end 1.33 -14.03) (layer "B.SilkS") (width 0.12))
+    (fp_line (start 1.8 1.8) (end -1.8 1.8) (layer "B.CrtYd") (width 0.05))
+    (fp_line (start -1.8 -14.5) (end 1.8 -14.5) (layer "B.CrtYd") (width 0.05))
+    (fp_line (start 1.8 -14.5) (end 1.8 1.8) (layer "B.CrtYd") (width 0.05))
+    (fp_line (start -1.8 1.8) (end -1.8 -14.5) (layer "B.CrtYd") (width 0.05))
+    (fp_line (start 1.27 -13.97) (end -1.27 -13.97) (layer "B.Fab") (width 0.1))
+    (fp_line (start 1.27 1.27) (end 1.27 -13.97) (layer "B.Fab") (width 0.1))
+    (fp_line (start -0.635 1.27) (end 1.27 1.27) (layer "B.Fab") (width 0.1))
+    (fp_line (start -1.27 -13.97) (end -1.27 0.635) (layer "B.Fab") (width 0.1))
+    (fp_line (start -1.27 0.635) (end -0.635 1.27) (layer "B.Fab") (width 0.1))
+    (pad "1" thru_hole rect locked (at 0 0 90) (size 1.7 1.7) (drill 1) (layers *.Cu *.Mask)
+      (net 1 "GND") (pinfunction "Pin_1") (pintype "passive"))
+    (pad "2" thru_hole oval locked (at 0 -2.54 90) (size 1.7 1.7) (drill 1) (layers *.Cu *.Mask)
+      (net 1 "GND") (pinfunction "Pin_2") (pintype "passive"))
+    (pad "3" thru_hole oval locked (at 0 -5.08 90) (size 1.7 1.7) (drill 1) (layers *.Cu *.Mask)
+      (net 62 "unconnected-(J2-Pad3)") (pinfunction "Pin_3") (pintype "passive+no_connect"))
+    (pad "4" thru_hole oval locked (at 0 -7.62 90) (size 1.7 1.7) (drill 1) (layers *.Cu *.Mask)
+      (net 61 "Net-(J2-Pad4)") (pinfunction "Pin_4") (pintype "passive"))
+    (pad "5" thru_hole oval locked (at 0 -10.16 90) (size 1.7 1.7) (drill 1) (layers *.Cu *.Mask)
+      (net 60 "Net-(J2-Pad5)") (pinfunction "Pin_5") (pintype "passive"))
+    (pad "6" thru_hole oval locked (at 0 -12.7 90) (size 1.7 1.7) (drill 1) (layers *.Cu *.Mask)
+      (net 8 "Net-(C7-Pad1)") (pinfunction "Pin_6") (pintype "passive"))
+    (model "${HPS3DMOD}/PinHeader_1x06_P2.54mm_Vertical.wrl"
+      (offset (xyz 0 0 0))
+      (scale (xyz 1 1 1))

Commit message: Update HPS_Round_Clock.kicad_pcb
Parts:
- moved C61 0.63 mm to (132.1, 75.6)
Routing:
- net GND: track 258.4 -> 259.2 mm
- net SCL: track 47.6 -> 48.2 mm
- net Net-(R4-Pad2): vias 2 -> 1
