File: HPS_Round_Clock/HPS_Round_Clock.kicad_pcb (KiCad board)
At the start: 2 copper layers, 118 x 118 mm, 149 parts, among them J1 Power_inlet_vertical, J2 Conn_01x06, SW1 Omron_B3F_SPST, SW2 Omron_B3F_SPST, SW3 Omron_B3F_SPST, SW4 Omron_B3F_SPST, SW5 Omron_B3F_SPST, U1 L7805, U2 DS1307_DIP-8, U4 ATmega328-PU, U5 TSOP38238, Y1 Crystal_16MHz, Y2 Crystal_32768Hz

Commit message: Update HPS_Round_Clock.kicad_pcb
Parts:
- removed TP10, TP9: TestPoint, footprints:TestPoint_THTPad_D2.0mm_Drill1.0mm
- removed U5: TSOP38238, footprints:Vishay_MINICAST-3Pin
- added D66: LED_0805, footprints:LED_0805_2012Metric, F.Cu at (149.9, 67.9)
- added J3: Conn_02x03_Odd_Even, footprints:PinHeader_2x03_P2.54mm_Vertical, F.Cu at (149.2, 81.9)
- added R10: R_0805_4.7K, footprints:R_0805_2012Metric, F.Cu at (123.2, 83.2)
- added R11: R_0805_4.7K, footprints:R_0805_2012Metric, F.Cu at (137.8, 71.8)
- added R8: R_0805_2.2K, footprints:R_0805_2012Metric, F.Cu at (149.9, 70.5)
- added U3: TSOP38238_Horiz, footprints:Vishay_MINICAST-3Pin_Horiz, F.Cu at (154.9, 93.2)
- moved R9 9.99 mm to (165.1, 94.0)
- moved C57 8.98 mm to (158.1, 71.1)
- moved D100 7.65 mm to (163.2, 90.2)
- moved TP11 5.85 mm to (160.7, 67.9)
- moved TP4 4.84 mm to (148.0, 61.6)
- moved C5 1.02 mm to (151.8, 92.1)
- moved R5 0.68 mm to (160.7, 139.1), turned to -162 degrees
- moved Y2 0.58 mm to (144.7, 83.2)
- moved U2 0.48 mm to (145.8, 85.7)
- moved R3 0.41 mm to (140.5, 139.3), turned to 162 degrees
- moved TP13 0.28 mm to (149.1, 90.4)
- moved TP12 0.25 mm to (149.2, 93.6)
- moved R4 0.25 mm to (151.1, 140.7), turned to 180 degrees
Connections:
- R1 pad 1: GND -> VCC
- R3 pad 1: GND -> Net-(R3-Pad1)
- R3 pad 2: Net-(R3-Pad2) -> VCC
- R4 pad 1: GND -> Net-(R4-Pad1)
- R4 pad 2: Net-(R4-Pad2) -> VCC
- R5 pad 1: GND -> Net-(R5-Pad1)
- R5 pad 2: Net-(R5-Pad2) -> VCC
- SW1 pad 3: VCC -> GND
- SW1 pad 4: VCC -> GND
- SW2 pad 1: Net-(R3-Pad2) -> Net-(R3-Pad1)
- SW2 pad 2: Net-(R3-Pad2) -> Net-(R3-Pad1)
- SW2 pad 3: VCC -> GND
- SW2 pad 4: VCC -> GND
- SW3 pad 1: Net-(R4-Pad2) -> Net-(R4-Pad1)
- SW3 pad 2: Net-(R4-Pad2) -> Net-(R4-Pad1)
- SW3 pad 3: VCC -> GND
- SW3 pad 4: VCC -> GND
- SW4 pad 1: Net-(R5-Pad2) -> Net-(R5-Pad1)
- SW4 pad 2: Net-(R5-Pad2) -> Net-(R5-Pad1)
- SW4 pad 3: VCC -> GND
- SW4 pad 4: VCC -> GND
- U4 pad 13: Net-(R5-Pad2) -> Net-(R5-Pad1)
- U4 pad 17: Net-(TP9-Pad1) -> MOSI
- U4 pad 18: Net-(TP10-Pad1) -> MISO
- U4 pad 5: Net-(R3-Pad2) -> Net-(R3-Pad1)
- U4 pad 6: Net-(R4-Pad2) -> Net-(R4-Pad1)
Routing:
- net Net-(R5-Pad2): track 47.8 -> 0.00 mm, vias 2 -> 0
- net Net-(R5-Pad1): track 0.00 -> 47.3 mm, vias 0 -> 2
- net Net-(R4-Pad2): track 40.9 -> 0.00 mm, vias 1 -> 0
- net Net-(R3-Pad2): track 40.0 -> 0.00 mm, vias 1 -> 0
- net Net-(R4-Pad1): track 0.00 -> 39.9 mm, vias 0 -> 1
- net Net-(R3-Pad1): track 0.00 -> 39.6 mm, vias 0 -> 1
- net Net-(TP9-Pad1): track 29.8 -> 0.00 mm, vias 1 -> 0
- net Net-(TP10-Pad1): track 29.5 -> 0.00 mm
- net MISO: track 0.00 -> 27.6 mm, vias 0 -> 1
- net MOSI: track 0.00 -> 23.4 mm, vias 0 -> 1
- net LED_SCK: track 0.00 -> 16.4 mm, vias 0 -> 1
- net RESET: track 73.9 -> 88.1 mm, vias 3 -> 4
- net GND: track 259.2 -> 271.1 mm, vias 113 -> 118
- net Net-(TP11-Pad1): track 30.8 -> 35.1 mm
- net Outer LED Ring: track 67.3 -> 71.0 mm
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
Commit message: Full Gerber Push
Parts:
- moved Y1 0.46 mm to (157.6, 108.2)
Other:
- board text added: "A"
- board text added: "E"
- board text added: "I"
- board text added: "M"
- board text added: "O"
- board text added: "T"
- board text added: "U"
Changed lines of the file:
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@@
     )
     (pad_to_mask_clearance 0)
+    (aux_axis_origin 91 159)
     (pcbplotparams
       (layerselection 0x00010fc_ffffffff)
@@
       (viasonmask false)
       (mode 1)
-      (useauxorigin false)
+      (useauxorigin true)
       (hpglpennumber 1)
       (hpglpenspeed 20)
@@
       (psa4output false)
       (plotreference true)
-      (plotvalue true)
+      (plotvalue false)
       (plotinvisibletext false)
       (sketchpadsonfab false)
-      (subtractmaskfromsilk false)
+      (subtractmaskfromsilk true)
       (outputformat 1)
       (mirror false)
       (drillshape 0)
       (scaleselection 1)
-      (outputdirectory "")
+      (outputdirectory "./")
     )
   )
@@
   )
   (footprint "footprints:Crystal_SMD_HC49-SD" (layer "F.Cu")
-    (at 158 107.95 180)
+    (at 157.619 108.204 180)
     (descr "SMD Crystal HC-49-SD http://cdn-reichelt.de/documents/datenblatt/B400/xxx-HC49-SMD.pdf, 11.4x4.7mm^2 package")
     (tags "SMD SMT crystal")
@@
   (gr_circle locked (center 150 100) (end 209 100) (layer "Edge.Cuts") (width 0.1) (fill none))
   (gr_circle locked (center 150 100) (end 150 50) (layer "User.4") (width 0.15) (fill none))
+  (gr_text "T" (at 104.775 69.85 56) (layer "F.SilkS")
+    (effects (font (size 5.08 5.08) (thickness 0.762)))
+  )
+  (gr_text "E" (at 136.525 47.625 13) (layer "F.SilkS")
+    (effects (font (size 5.08 5.08) (thickness 0.762)))
+  )
+  (gr_text "T" (at 115.57 57.785 40) (layer "F.SilkS")
+    (effects (font (size 5.08 5.08) (thickness 0.762)))
+  )
+  (gr_text "A" (at 109.22 63.5 48) (layer "F.SilkS")
+    (effects (font (size 5.08 5.08) (thickness 0.762)))
+  )
+  (gr_text "M" (at 128.905 50.165 24) (layer "F.SilkS")
+    (effects (font (size 5.08 5.08) (thickness 0.762)))
+  )
+  (gr_text "U" (at 100.33 77.47 68) (layer "F.SilkS")
+    (effects (font (size 5.08 5.08) (thickness 0.762)))
+  )
+  (gr_text "I" (at 121.92 53.34 32) (layer "F.SilkS")
+    (effects (font (size 5.08 5.08) (thickness 0.762)))
+  )
+  (gr_text "O" (at 96.52 86.995 261) (layer "F.SilkS")
+    (effects (font (size 5.08 5.08) (thickness 0.762)))
+  )
   (segment (start 145.2 127) (end 143.51 127) (width 0.2032) (layer "F.Cu") (net 1))
   (segment (start 198.472342 86.712342) (end 198.755 86.995) (width 0.2032) (layer "F.Cu") (net 1))
@@
   (segment (start 192.405 73.66) (end 193.04 73.66) (width 0.2032) (layer "F.Cu") (net 1))
   (segment (start 102.873779 110.176904) (end 101.278096 110.176904) (width 0.2032) (layer "F.Cu") (net 1))
-  (segment (start 150.28 109.855) (end 149.225 108.8) (width 0.2032) (layer "F.Cu") (net 1))
   (segment (start 127 111.481087) (end 127 111.125) (width 0.2032) (layer "F.Cu") (net 1))
   (segment (start 191.77 126.400197) (end 191.77 128.27) (width 0.2032) (layer "F.Cu") (net 1))
@@
   (segment (start 121.111602 88.438398) (end 121.285 88.265) (width 0.2032) (layer "F.Cu") (net 1))
   (segment (start 169.791429 130.913551) (end 170.957878 132.08) (width 0.2032) (layer "F.Cu") (net 1))
+  (segment (start 149.225 110.49) (end 149.225 108.8) (width 0.2032) (layer "F.Cu") (net 1))
   (segment (start 110.959969 71.813217) (end 109.631752 70.485) (width 0.2032) (layer "F.Cu") (net 1))
   (segment (start 182.565078 109.534922) (end 183.515 108.585) (width 0.2032) (layer "F.Cu") (net 1))
@@
   (segment (start 167.64 123.19) (end 167.64 125.095) (width 0.2032) (layer "F.Cu") (net 1))
   (segment (start 160.917664 151.938398) (end 159.846602 151.938398) (width 0.2032) (layer "F.Cu") (net 1))
-  (segment (start 150.495 109.855) (end 150.28 109.855) (width 0.2032) (layer "F.Cu") (net 1))
   (segment (start 148.9225 67.945) (end 147.32 67.945) (width 0.2032) (layer "F.Cu") (net 1))
   (segment (start 142.875 149.86) (end 143.200778 149.86) (width 0.2032) (layer "F.Cu") (net 1))
@@
   (via (at 186.69 88.265) (size 0.8128) (drill 0.4064) (layers "F.Cu" "B.Cu") (net 1))
   (via (at 182.245 138.43) (size 0.8128) (drill 0.4064) (layers "F.Cu" "B.Cu") (net 1))
-  (via (at 150.495 109.855) (size 0.8128) (drill 0.4064) (layers "F.Cu" "B.Cu") (net 1))
+  (via (at 149.225 110.49) (size 0.8128) (drill 0.4064) (layers "F.Cu" "B.Cu") (net 1))
   (via (at 180.34 105.41) (size 0.8128) (drill 0.4064) (layers "F.Cu" "B.Cu") (net 1))
   (via (at 200.025 107.315) (size 0.8128) (drill 0.4064) (layers "F.Cu" "B.Cu") (net 1))
