File: HPS_Round_Clock/untitled.kicad_sch (KiCad schematic)
At the start: 22 parts

Commit message: Update untitled.kicad_sch
Parts:
- removed C13, C14: C_0805_0.1uf, footprints:C_0805_2012Metric, symbol HPS:C_0805_0.1uf
Changed lines of the file:
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@@
   (junction (at 142.24 85.09) (diameter 0) (color 0 0 0 0)
   )
-  (junction (at 203.2 85.09) (diameter 0) (color 0 0 0 0)
-  )
   (junction (at 162.56 62.23) (diameter 0) (color 0 0 0 0)
   )
@@
   (junction (at 121.92 22.86) (diameter 0) (color 0 0 0 0)
   )
-  (junction (at 203.2 45.72) (diameter 0) (color 0 0 0 0)
-  )
   (junction (at 142.24 45.72) (diameter 0) (color 0 0 0 0)
   )
@@
   (junction (at 203.2 62.23) (diameter 0) (color 0 0 0 0)
   )
-  (junction (at 231.14 22.86) (diameter 0) (color 0 0 0 0)
-  )
   (junction (at 142.24 62.23) (diameter 0) (color 0 0 0 0)
   )
@@
   )
   (junction (at 121.92 45.72) (diameter 0) (color 0 0 0 0)
-  )
-  (junction (at 231.14 62.23) (diameter 0) (color 0 0 0 0)
   )
   (junction (at 60.96 85.09) (diameter 0) (color 0 0 0 0)
@@
     (stroke (width 0) (type default) (color 0 0 0 0))
   )
-  (wire (pts (xy 203.2 85.09) (xy 231.14 85.09))
-    (stroke (width 0) (type default) (color 0 0 0 0))
-  )
   (wire (pts (xy 182.88 85.09) (xy 203.2 85.09))
     (stroke (width 0) (type default) (color 0 0 0 0))
@@
     (stroke (width 0) (type default) (color 0 0 0 0))
   )
-  (wire (pts (xy 231.14 62.23) (xy 231.14 69.85))
-    (stroke (width 0) (type default) (color 0 0 0 0))
-  )
   (wire (pts (xy 142.24 22.86) (xy 162.56 22.86))
     (stroke (width 0) (type default) (color 0 0 0 0))
@@
     (stroke (width 0) (type default) (color 0 0 0 0))
   )
-  (wire (pts (xy 231.14 38.1) (xy 231.14 45.72))
-    (stroke (width 0) (type default) (color 0 0 0 0))
-  )
   (wire (pts (xy 78.74 36.83) (xy 83.82 36.83))
     (stroke (width 0) (type default) (color 0 0 0 0))
@@
     (stroke (width 0) (type default) (color 0 0 0 0))
   )
-  (wire (pts (xy 231.14 77.47) (xy 231.14 85.09))
-    (stroke (width 0) (type default) (color 0 0 0 0))
-  )
   (wire (pts (xy 121.92 40.64) (xy 121.92 45.72))
     (stroke (width 0) (type default) (color 0 0 0 0))
@@
     (stroke (width 0) (type default) (color 0 0 0 0))
   )
-  (wire (pts (xy 203.2 45.72) (xy 231.14 45.72))
-    (stroke (width 0) (type default) (color 0 0 0 0))
-  )
   (wire (pts (xy 38.1 76.2) (xy 43.18 76.2))
     (stroke (width 0) (type default) (color 0 0 0 0))
@@
   )
   (wire (pts (xy 60.96 40.64) (xy 60.96 45.72))
-    (stroke (width 0) (type default) (color 0 0 0 0))
-  )
-  (wire (pts (xy 231.14 22.86) (xy 231.14 30.48))
     (stroke (width 0) (type default) (color 0 0 0 0))
   )
@@
     (pin "4")
   )
-  (symbol (lib_id "HPS:C_0805_0.1uf") (at 231.14 73.66 0) (unit 1)
-    (in_bom yes) (on_board yes) (fields_autoplaced)
-    (property "Reference" "C14" (id 0) (at 234.95 72.3899 0)
-      (effects (font (size 1.27 1.27)) (justify left))
-    )
-    (property "Value" "C_0805_0.1uf" (id 1) (at 234.95 74.9299 0)
-      (effects (font (size 1.27 1.27)) (justify left))
-    )
-    (property "Footprint" "footprints:C_0805_2012Metric" (id 2) (at 232.1052 77.47 0)
-      (effects (font (size 1.27 1.27)) hide)
-    )
-    (property "Datasheet" "https://datasheets.avx.com/X7RDielectric.pdf" (id 3) (at 231.775 71.12 0)
-      (effects (font (size 1.27 1.27)) hide)
-    )
-    (property "MFG" "AVX Corporation" (id 4) (at 231.14 80.01 0)
-      (effects (font (size 1.27 1.27)) hide)
-    )
-    (property "MPN" "08055C104KAT2A" (id 5) (at 231.14 82.55 0)
-      (effects (font (size 1.27 1.27)) hide)
-    )
-    (property "Digikey PN" "478-1395-1-ND" (id 6) (at 231.14 87.63 0)
-      (effects (font (size 1.27 1.27)) hide)
-    )
-    (property "Mouser PN" "N/A" (id 7) (at 231.14 90.17 0)
-      (effects (font (size 1.27 1.27)) hide)
-    )
-    (property "Voltage" "N/A" (id 8) (at 231.14 92.71 0)
-      (effects (font (size 1.27 1.27)) hide)
-    )
-    (property "Dielectric" "N/A" (id 9) (at 231.14 92.71 0)
-      (effects (font (size 1.27 1.27)) hide)
-    )
-    (property "Tolerance" "N/A" (id 10) (at 231.14 92.71 0)
-      (effects (font (size 1.27 1.27)) hide)
-    )
-    (pin "1")
-    (pin "2")
-  )
   (symbol (lib_id "HPS:NEOPIXEL_SMT") (at 71.12 36.83 0) (unit 1)
     (in_bom yes) (on_board yes) (fields_autoplaced)
@@
     (pin "4")
   )
-  (symbol (lib_id "HPS:C_0805_0.1uf") (at 231.14 34.29 0) (unit 1)
-    (in_bom yes) (on_board yes) (fields_autoplaced)
-    (property "Reference" "C13" (id 0) (at 234.95 33.0199 0)
-      (effects (font (size 1.27 1.27)) (justify left))
-    )
-    (property "Value" "C_0805_0.1uf" (id 1) (at 234.95 35.5599 0)
-      (effects (font (size 1.27 1.27)) (justify left))
-    )
-    (property "Footprint" "footprints:C_0805_2012Metric" (id 2) (at 232.1052 38.1 0)
-      (effects (font (size 1.27 1.27)) hide)
-    )
-    (property "Datasheet" "https://datasheets.avx.com/X7RDielectric.pdf" (id 3) (at 231.775 31.75 0)
-      (effects (font (size 1.27 1.27)) hide)
-    )
-    (property "MFG" "AVX Corporation" (id 4) (at 231.14 40.64 0)
-      (effects (font (size 1.27 1.27)) hide)
-    )
-    (property "MPN" "08055C104KAT2A" (id 5) (at 231.14 43.18 0)
-      (effects (font (size 1.27 1.27)) hide)
-    )
-    (property "Digikey PN" "478-1395-1-ND" (id 6) (at 231.14 48.26 0)
-      (effects (font (size 1.27 1.27)) hide)
-    )
-    (property "Mouser PN" "N/A" (id 7) (at 231.14 50.8 0)
-      (effects (font (size 1.27 1.27)) hide)
-    )
-    (property "Voltage" "N/A" (id 8) (at 231.14 53.34 0)
-      (effects (font (size 1.27 1.27)) hide)
-    )
-    (property "Dielectric" "N/A" (id 9) (at 231.14 53.34 0)
-      (effects (font (size 1.27 1.27)) hide)
-    )
-    (property "Tolerance" "N/A" (id 10) (at 231.14 53.34 0)
-      (effects (font (size 1.27 1.27)) hide)
-    )
-    (pin "1")
-    (pin "2")
-  )
   (symbol (lib_id "HPS:GND") (at 17.78 48.26 0) (unit 1)
